Commit message: 🐞 fix(RL环境): 构型展示流程
加速训练，解决不同构型切换后产生的bug

File: test/urdf/unit7.urdf (robot description, URDF)
Before this commit: robot UNNAMED_0, 41 links, 40 joints
Links:
- removed link BLM1_BLU10_BLU10_BLU10_BLU10_BLU10_BLU10_BLU10_BLU10_BLU10_BLU10_BLU10_BLU10_BLU10_BLU10_BLU10_BLU10_BLU10_BLU10_BLU10_BLU10_BLU10_U_b_body
- removed link BLM1_BLU10_BLU10_BLU10_BLU10_BLU10_BLU10_BLU10_BLU10_BLU10_BLU10_BLU10_BLU10_BLU10_BLU10_BLU10_BLU10_BLU10_BLU10_BLU10_BLU10_BLU10_U_b_in
- removed link BLM1_BLU10_BLU10_BLU10_BLU10_BLU10_BLU10_BLU10_BLU10_BLU10_BLU10_BLU10_BLU10_BLU10_BLU10_BLU10_BLU10_BLU10_BLU10_BLU10_BLU10_ILU33_U_ci_body
- removed link BLM1_BLU10_BLU10_BLU10_BLU10_BLU10_BLU10_BLU10_BLU10_BLU10_BLU10_BLU10_BLU10_BLU10_BLU10_BLU10_BLU10_BLU10_BLU10_BLU10_BLU10_ILU33_U_ci_in
- removed link BLM1_BLU10_BLU10_BLU10_BLU10_BLU10_BLU10_BLU10_BLU10_BLU10_BLU10_BLU10_BLU10_BLU10_BLU10_BLU10_BLU10_BLU10_BLU10_BLU10_JTLU18_U_tj_body
- removed link BLM1_BLU10_BLU10_BLU10_BLU10_BLU10_BLU10_BLU10_BLU10_BLU10_BLU10_BLU10_BLU10_BLU10_BLU10_BLU10_BLU10_BLU10_BLU10_BLU10_JTLU18_U_tj_in
- removed link BLM1_BLU10_BLU10_BLU10_BLU10_BLU10_BLU10_BLU10_BLU10_BLU10_BLU10_BLU10_BLU10_BLU10_BLU10_BLU10_BLU10_BLU10_BLU10_ILU34_U_ci_body
- removed link BLM1_BLU10_BLU10_BLU10_BLU10_BLU10_BLU10_BLU10_BLU10_BLU10_BLU10_BLU10_BLU10_BLU10_BLU10_BLU10_BLU10_BLU10_BLU10_ILU34_U_ci_in
- removed link BLM1_BLU10_BLU10_BLU10_BLU10_BLU10_BLU10_BLU10_BLU10_BLU10_BLU10_BLU10_BLU10_BLU10_BLU10_BLU10_BLU10_BLU10_JTLU19_U_tj_body
- removed link BLM1_BLU10_BLU10_BLU10_BLU10_BLU10_BLU10_BLU10_BLU10_BLU10_BLU10_BLU10_BLU10_BLU10_BLU10_BLU10_BLU10_BLU10_JTLU19_U_tj_in
- removed link BLM1_BLU10_BLU10_BLU10_BLU10_BLU10_BLU10_BLU10_BLU10_BLU10_BLU10_BLU10_BLU10_BLU10_BLU10_BLU10_BLU10_ILU35_U_ci_body
- removed link BLM1_BLU10_BLU10_BLU10_BLU10_BLU10_BLU10_BLU10_BLU10_BLU10_BLU10_BLU10_BLU10_BLU10_BLU10_BLU10_BLU10_ILU35_U_ci_in
- removed link BLM1_BLU10_BLU10_BLU10_BLU10_BLU10_BLU10_BLU10_BLU10_BLU10_BLU10_BLU10_BLU10_BLU10_BLU10_BLU10_SLMU8_U_sl_body
- removed link BLM1_BLU10_BLU10_BLU10_BLU10_BLU10_BLU10_BLU10_BLU10_BLU10_BLU10_BLU10_BLU10_BLU10_BLU10_IMU26_U_reverse_U_ic_body
- removed link BLM1_BLU10_BLU10_BLU10_BLU10_BLU10_BLU10_BLU10_BLU10_BLU10_BLU10_BLU10_BLU10_BLU10_BLU10_IMU26_U_reverse_U_ic_in
- removed link BLM1_BLU10_BLU10_BLU10_BLU10_BLU10_BLU10_BLU10_BLU10_BLU10_BLU10_BLU10_BLU10_BLU10_JTMU9_U_reverse_U_tj_body
- removed link BLM1_BLU10_BLU10_BLU10_BLU10_BLU10_BLU10_BLU10_BLU10_BLU10_BLU10_BLU10_BLU10_BLU10_JTMU9_U_reverse_U_tj_in
- removed link BLM1_BLU10_BLU10_BLU10_BLU10_BLU10_BLU10_BLU10_BLU10_BLU10_BLU10_BLU10_BLU10_IMU27_reverse_IMU27_U_ic_body
- removed link BLM1_BLU10_BLU10_BLU10_BLU10_BLU10_BLU10_BLU10_BLU10_BLU10_BLU10_BLU10_BLU10_IMU27_reverse_IMU27_U_ic_in
- removed link BLM1_BLU10_BLU10_BLU10_BLU10_BLU10_BLU10_BLU10_BLU10_BLU10_BLU10_BLU10_CMMU6_U_cl_body
- removed link BLM1_BLU10_BLU10_BLU10_BLU10_BLU10_BLU10_BLU10_BLU10_BLU10_BLU10_BLU10_CMMU6_U_cl_in_1
- removed link BLM1_BLU10_BLU10_BLU10_BLU10_BLU10_BLU10_BLU10_BLU10_BLU10_BLU10_BLU10_CMMU6_U_cl_in_2
- removed link BLM1_BLU10_BLU10_BLU10_BLU10_BLU10_BLU10_BLU10_BLU10_BLU10_BLU10_IMU28_U_ic_body
- removed link BLM1_BLU10_BLU10_BLU10_BLU10_BLU10_BLU10_BLU10_BLU10_BLU10_BLU10_IMU28_U_ic_in
- removed link BLM1_BLU10_BLU10_BLU10_BLU10_BLU10_BLU10_BLU10_BLU10_BLU10_SMSU5_U_sl_body
- removed link BLM1_BLU10_BLU10_BLU10_BLU10_BLU10_BLU10_BLU10_BLU10_ISU15_U_reverse_U_ic_body
- removed link BLM1_BLU10_BLU10_BLU10_BLU10_BLU10_BLU10_BLU10_BLU10_ISU15_U_reverse_U_ic_in
- removed link BLM1_BLU10_BLU10_BLU10_BLU10_BLU10_BLU10_BLU10_JSU13_U_reverse_U_tj_body
- removed link BLM1_BLU10_BLU10_BLU10_BLU10_BLU10_BLU10_BLU10_JSU13_U_reverse_U_tj_in
- removed link BLM1_BLU10_BLU10_BLU10_BLU10_BLU10_BLU10_ISU16_U_reverse_U_ic_body
- removed link BLM1_BLU10_BLU10_BLU10_BLU10_BLU10_BLU10_ISU16_U_reverse_U_ic_in
- removed link BLM1_BLU10_BLU10_BLU10_BLU10_BLU10_JSU14_U_reverse_U_tj_body
- removed link BLM1_BLU10_BLU10_BLU10_BLU10_BLU10_JSU14_U_reverse_U_tj_in
- removed link BLM1_BLU10_BLU10_BLU10_BLU10_ISU17_U_reverse_U_ic_body
- removed link BLM1_BLU10_BLU10_BLU10_BLU10_ISU17_U_reverse_U_ic_in
- removed link BLM1_BLU10_BLU10_BLU10_JSU15_U_reverse_U_tj_body
- removed link BLM1_BLU10_BLU10_BLU10_JSU15_U_reverse_U_tj_in
- removed link BLM1_BLU10_BLU10_ISU18_reverse_ISU18_U_ic_body
- removed link BLM1_BLU10_BLU10_ISU18_reverse_ISU18_U_ic_in
- removed link BLM1_BLU10_ESU1_U_e_body
- removed link BLM1_BLU10_ESU1_U_e_in
- added link BLM1_BLU65_BLU65_BLU65_BLU65_BLU65_BLU65_BLU65_BLU65_BLU65_BLU65_BLU65_BLU65_BLU65_BLU65_BLU65_BLU65_BLU65_BLU65_BLU65_BLU65_BLU65_U_b_body, mass 0; collision mesh filename=package://base-l.SLDASM/meshes/b_body.STL; visual mesh filename=package://base-l.SLDASM/meshes/b_body.STL
- added link BLM1_BLU65_BLU65_BLU65_BLU65_BLU65_BLU65_BLU65_BLU65_BLU65_BLU65_BLU65_BLU65_BLU65_BLU65_BLU65_BLU65_BLU65_BLU65_BLU65_BLU65_BLU65_U_b_in, mass 5.9754; collision mesh filename=package://base-l.SLDASM/meshes/b_in.STL; visual mesh filename=package://base-l.SLDASM/meshes/b_in.STL
- added link BLM1_BLU65_BLU65_BLU65_BLU65_BLU65_BLU65_BLU65_BLU65_BLU65_BLU65_BLU65_BLU65_BLU65_BLU65_BLU65_BLU65_BLU65_BLU65_BLU65_BLU65_ILU188_U_ci_body, mass 0; collision mesh filename=package://input_connector_l.SLDASM/meshes/ci_body.STL; visual mesh filename=package://input_connector_l.SLDASM/meshes/ci_body.STL
- added link BLM1_BLU65_BLU65_BLU65_BLU65_BLU65_BLU65_BLU65_BLU65_BLU65_BLU65_BLU65_BLU65_BLU65_BLU65_BLU65_BLU65_BLU65_BLU65_BLU65_BLU65_ILU188_U_ci_in, mass 0; collision mesh filename=package://input_connector_l.SLDASM/meshes/ci_in.STL; visual mesh filename=package://input_connector_l.SLDASM/meshes/ci_in.STL
- added link BLM1_BLU65_BLU65_BLU65_BLU65_BLU65_BLU65_BLU65_BLU65_BLU65_BLU65_BLU65_BLU65_BLU65_BLU65_BLU65_BLU65_BLU65_BLU65_BLU65_JTLU118_U_tj_body, mass 1.5884; collision mesh filename=package://jointT-l.SLDASM/meshes/tj_body.STL; visual mesh filename=package://jointT-l.SLDASM/meshes/tj_body.STL
- added link BLM1_BLU65_BLU65_BLU65_BLU65_BLU65_BLU65_BLU65_BLU65_BLU65_BLU65_BLU65_BLU65_BLU65_BLU65_BLU65_BLU65_BLU65_BLU65_BLU65_JTLU118_U_tj_in, mass 1.5884; collision mesh filename=package://jointT-l.SLDASM/meshes/tj_in.STL; visual mesh filename=package://jointT-l.SLDASM/meshes/tj_in.STL
- added link BLM1_BLU65_BLU65_BLU65_BLU65_BLU65_BLU65_BLU65_BLU65_BLU65_BLU65_BLU65_BLU65_BLU65_BLU65_BLU65_BLU65_BLU65_BLU65_ILU189_U_ci_body, mass 0; collision mesh filename=package://input_connector_l.SLDASM/meshes/ci_body.STL; visual mesh filename=package://input_connector_l.SLDASM/meshes/ci_body.STL
- added link BLM1_BLU65_BLU65_BLU65_BLU65_BLU65_BLU65_BLU65_BLU65_BLU65_BLU65_BLU65_BLU65_BLU65_BLU65_BLU65_BLU65_BLU65_BLU65_ILU189_U_ci_in, mass 0; collision mesh filename=package://input_connector_l.SLDASM/meshes/ci_in.STL; visual mesh filename=package://input_connector_l.SLDASM/meshes/ci_in.STL
- added link BLM1_BLU65_BLU65_BLU65_BLU65_BLU65_BLU65_BLU65_BLU65_BLU65_BLU65_BLU65_BLU65_BLU65_BLU65_BLU65_BLU65_BLU65_JTLU119_U_tj_body, mass 1.5884; collision mesh filename=package://jointT-l.SLDASM/meshes/tj_body.STL; visual mesh filename=package://jointT-l.SLDASM/meshes/tj_body.STL
- added link BLM1_BLU65_BLU65_BLU65_BLU65_BLU65_BLU65_BLU65_BLU65_BLU65_BLU65_BLU65_BLU65_BLU65_BLU65_BLU65_BLU65_BLU65_JTLU119_U_tj_in, mass 1.5884; collision mesh filename=package://jointT-l.SLDASM/meshes/tj_in.STL; visual mesh filename=package://jointT-l.SLDASM/meshes/tj_in.STL
- added link BLM1_BLU65_BLU65_BLU65_BLU65_BLU65_BLU65_BLU65_BLU65_BLU65_BLU65_BLU65_BLU65_BLU65_BLU65_BLU65_BLU65_ILU190_U_ci_body, mass 0; collision mesh filename=package://input_connector_l.SLDASM/meshes/ci_body.STL; visual mesh filename=package://input_connector_l.SLDASM/meshes/ci_body.STL
- added link BLM1_BLU65_BLU65_BLU65_BLU65_BLU65_BLU65_BLU65_BLU65_BLU65_BLU65_BLU65_BLU65_BLU65_BLU65_BLU65_BLU65_ILU190_U_ci_in, mass 0; collision mesh filename=package://input_connector_l.SLDASM/meshes/ci_in.STL; visual mesh filename=package://input_connector_l.SLDASM/meshes/ci_in.STL
- added link BLM1_BLU65_BLU65_BLU65_BLU65_BLU65_BLU65_BLU65_BLU65_BLU65_BLU65_BLU65_BLU65_BLU65_BLU65_BLU65_SLMU44_U_sl_body, mass 1.4196; collision mesh filename=package://straight_link-lm.SLDASM/meshes/sl_body.STL; visual mesh filename=package://straight_link-lm.SLDASM/meshes/sl_body.STL
- added link BLM1_BLU65_BLU65_BLU65_BLU65_BLU65_BLU65_BLU65_BLU65_BLU65_BLU65_BLU65_BLU65_BLU65_BLU65_IMU96_U_reverse_U_ic_body, mass 0; collision mesh filename=package://input_connector_m.SLDASM/meshes/ic_body.STL; visual mesh filename=package://input_connector_m.SLDASM/meshes/ic_body.STL
- added link BLM1_BLU65_BLU65_BLU65_BLU65_BLU65_BLU65_BLU65_BLU65_BLU65_BLU65_BLU65_BLU65_BLU65_BLU65_IMU96_U_reverse_U_ic_in, mass 0.50882; collision mesh filename=package://input_connector_m.SLDASM/meshes/ic_in.STL; visual mesh filename=package://input_connector_m.SLDASM/meshes/ic_in.STL
- added link BLM1_BLU65_BLU65_BLU65_BLU65_BLU65_BLU65_BLU65_BLU65_BLU65_BLU65_BLU65_BLU65_BLU65_JTMU37_U_reverse_U_tj_body, mass 0.93065; collision mesh filename=package://jointT-m.SLDASM/meshes/tj_body.STL; visual mesh filename=package://jointT-m.SLDASM/meshes/tj_body.STL
- added link BLM1_BLU65_BLU65_BLU65_BLU65_BLU65_BLU65_BLU65_BLU65_BLU65_BLU65_BLU65_BLU65_BLU65_JTMU37_U_reverse_U_tj_in, mass 0.93066; collision mesh filename=package://jointT-m.SLDASM/meshes/tj_in.STL; visual mesh filename=package://jointT-m.SLDASM/meshes/tj_in.STL
- added link BLM1_BLU65_BLU65_BLU65_BLU65_BLU65_BLU65_BLU65_BLU65_BLU65_BLU65_BLU65_BLU65_IMU97_reverse_IMU97_U_ic_body, mass 0; collision mesh filename=package://input_connector_m.SLDASM/meshes/ic_body.STL; visual mesh filename=package://input_connector_m.SLDASM/meshes/ic_body.STL
- added link BLM1_BLU65_BLU65_BLU65_BLU65_BLU65_BLU65_BLU65_BLU65_BLU65_BLU65_BLU65_BLU65_IMU97_reverse_IMU97_U_ic_in, mass 0.50882; collision mesh filename=package://input_connector_m.SLDASM/meshes/ic_in.STL; visual mesh filename=package://input_connector_m.SLDASM/meshes/ic_in.STL
- added link BLM1_BLU65_BLU65_BLU65_BLU65_BLU65_BLU65_BLU65_BLU65_BLU65_BLU65_BLU65_CMMU27_U_cl_body, mass 0.93065; collision mesh filename=package://corner_link-mm.SLDASM/meshes/cl_body.STL; visual mesh filename=package://corner_link-mm.SLDASM/meshes/cl_body.STL
- added link BLM1_BLU65_BLU65_BLU65_BLU65_BLU65_BLU65_BLU65_BLU65_BLU65_BLU65_BLU65_CMMU27_U_cl_in_1, mass 0.93066; collision mesh filename=package://corner_link-mm.SLDASM/meshes/cl_in_1.STL; visual mesh filename=package://corner_link-mm.SLDASM/meshes/cl_in_1.STL
- added link BLM1_BLU65_BLU65_BLU65_BLU65_BLU65_BLU65_BLU65_BLU65_BLU65_BLU65_BLU65_CMMU27_U_cl_in_2, mass 0.93066; collision mesh filename=package://corner_link-mm.SLDASM/meshes/cl_in_2.STL; visual mesh filename=package://corner_link-mm.SLDASM/meshes/cl_in_2.STL
- added link BLM1_BLU65_BLU65_BLU65_BLU65_BLU65_BLU65_BLU65_BLU65_BLU65_BLU65_IMU98_U_ic_body, mass 0; collision mesh filename=package://input_connector_m.SLDASM/meshes/ic_body.STL; visual mesh filename=package://input_connector_m.SLDASM/meshes/ic_body.STL
- added link BLM1_BLU65_BLU65_BLU65_BLU65_BLU65_BLU65_BLU65_BLU65_BLU65_BLU65_IMU98_U_ic_in, mass 0.50882; collision mesh filename=package://input_connector_m.SLDASM/meshes/ic_in.STL; visual mesh filename=package://input_connector_m.SLDASM/meshes/ic_in.STL
- added link BLM1_BLU65_BLU65_BLU65_BLU65_BLU65_BLU65_BLU65_BLU65_BLU65_SMSU20_U_sl_body, mass 0.86346; collision mesh filename=package://straight_link-ms.SLDASM/meshes/sl_body.STL; visual mesh filename=package://straight_link-ms.SLDASM/meshes/sl_body.STL
- added link BLM1_BLU65_BLU65_BLU65_BLU65_BLU65_BLU65_BLU65_BLU65_ISU35_U_reverse_U_ic_body, mass 0; collision mesh filename=package://input_connector_s.SLDASM/meshes/ic_body.STL; visual mesh filename=package://input_connector_s.SLDASM/meshes/ic_body.STL
- added link BLM1_BLU65_BLU65_BLU65_BLU65_BLU65_BLU65_BLU65_BLU65_ISU35_U_reverse_U_ic_in, mass 0.23832; collision mesh filename=package://input_connector_s.SLDASM/meshes/ic_in.STL; visual mesh filename=package://input_connector_s.SLDASM/meshes/ic_in.STL
- added link BLM1_BLU65_BLU65_BLU65_BLU65_BLU65_BLU65_BLU65_JSU32_U_reverse_U_tj_body, mass 0.50441; collision mesh filename=package://jointT-s.SLDASM/meshes/tj_body.STL; visual mesh filename=package://jointT-s.SLDASM/meshes/tj_body.STL
- added link BLM1_BLU65_BLU65_BLU65_BLU65_BLU65_BLU65_BLU65_JSU32_U_reverse_U_tj_in, mass 0.50441; collision mesh filename=package://jointT-s.SLDASM/meshes/tj_in.STL; visual mesh filename=package://jointT-s.SLDASM/meshes/tj_in.STL
- added link BLM1_BLU65_BLU65_BLU65_BLU65_BLU65_BLU65_ISU36_U_reverse_U_ic_body, mass 0; collision mesh filename=package://input_connector_s.SLDASM/meshes/ic_body.STL; visual mesh filename=package://input_connector_s.SLDASM/meshes/ic_body.STL
- added link BLM1_BLU65_BLU65_BLU65_BLU65_BLU65_BLU65_ISU36_U_reverse_U_ic_in, mass 0.23832; collision mesh filename=package://input_connector_s.SLDASM/meshes/ic_in.STL; visual mesh filename=package://input_connector_s.SLDASM/meshes/ic_in.STL
- added link BLM1_BLU65_BLU65_BLU65_BLU65_BLU65_JSU33_U_reverse_U_tj_body, mass 0.50441; collision mesh filename=package://jointT-s.SLDASM/meshes/tj_body.STL; visual mesh filename=package://jointT-s.SLDASM/meshes/tj_body.STL
- added link BLM1_BLU65_BLU65_BLU65_BLU65_BLU65_JSU33_U_reverse_U_tj_in, mass 0.50441; collision mesh filename=package://jointT-s.SLDASM/meshes/tj_in.STL; visual mesh filename=package://jointT-s.SLDASM/meshes/tj_in.STL
- added link BLM1_BLU65_BLU65_BLU65_BLU65_ISU37_U_reverse_U_ic_body, mass 0; collision mesh filename=package://input_connector_s.SLDASM/meshes/ic_body.STL; visual mesh filename=package://input_connector_s.SLDASM/meshes/ic_body.STL
- added link BLM1_BLU65_BLU65_BLU65_BLU65_ISU37_U_reverse_U_ic_in, mass 0.23832; collision mesh filename=package://input_connector_s.SLDASM/meshes/ic_in.STL; visual mesh filename=package://input_connector_s.SLDASM/meshes/ic_in.STL
- added link BLM1_BLU65_BLU65_BLU65_JSU34_U_reverse_U_tj_body, mass 0.50441; collision mesh filename=package://jointT-s.SLDASM/meshes/tj_body.STL; visual mesh filename=package://jointT-s.SLDASM/meshes/tj_body.STL
- added link BLM1_BLU65_BLU65_BLU65_JSU34_U_reverse_U_tj_in, mass 0.50441; collision mesh filename=package://jointT-s.SLDASM/meshes/tj_in.STL; visual mesh filename=package://jointT-s.SLDASM/meshes/tj_in.STL
- added link BLM1_BLU65_BLU65_ISU38_reverse_ISU38_U_ic_body, mass 0; collision mesh filename=package://input_connector_s.SLDASM/meshes/ic_body.STL; visual mesh filename=package://input_connector_s.SLDASM/meshes/ic_body.STL
- added link BLM1_BLU65_BLU65_ISU38_reverse_ISU38_U_ic_in, mass 0.23832; collision mesh filename=package://input_connector_s.SLDASM/meshes/ic_in.STL; visual mesh filename=package://input_connector_s.SLDASM/meshes/ic_in.STL
- added link BLM1_BLU65_ESU2_U_ee_body, mass 0.0019211; collision mesh filename=package://end_effector_v_s.SLDASM/meshes/ee_body.STL; visual mesh filename=package://end_effector_v_s.SLDASM/meshes/ee_body.STL
- added link BLM1_BLU65_ESU2_U_ee_in, mass 0.0019211; collision mesh filename=package://end_effector_v_s.SLDASM/meshes/ee_in.STL; visual mesh filename=package://end_effector_v_s.SLDASM/meshes/ee_in.STL
Joints:
- removed joint BLM1_BLU10_BLU10_BLU10_BLU10_BLU10_BLU10_BLU10_BLU10_BLU10_BLU10_BLU10_BLU10_BLU10_BLU10_BLU10_BLU10_BLU10_BLU10_BLU10_BLU10_BLU10_U_b_large
- removed joint BLM1_BLU10_BLU10_BLU10_BLU10_BLU10_BLU10_BLU10_BLU10_BLU10_BLU10_BLU10_BLU10_BLU10_BLU10_BLU10_BLU10_BLU10_BLU10_BLU10_BLU10_ILU33_U_ci_large_1
- removed joint BLM1_BLU10_BLU10_BLU10_BLU10_BLU10_BLU10_BLU10_BLU10_BLU10_BLU10_BLU10_BLU10_BLU10_BLU10_BLU10_BLU10_BLU10_BLU10_BLU10_BLU10_ILU33_U_ci_large_2
- removed joint BLM1_BLU10_BLU10_BLU10_BLU10_BLU10_BLU10_BLU10_BLU10_BLU10_BLU10_BLU10_BLU10_BLU10_BLU10_BLU10_BLU10_BLU10_BLU10_BLU10_JTLU18_U_tj_large_1
- removed joint BLM1_BLU10_BLU10_BLU10_BLU10_BLU10_BLU10_BLU10_BLU10_BLU10_BLU10_BLU10_BLU10_BLU10_BLU10_BLU10_BLU10_BLU10_BLU10_BLU10_JTLU18_U_tj_large_2
- removed joint BLM1_BLU10_BLU10_BLU10_BLU10_BLU10_BLU10_BLU10_BLU10_BLU10_BLU10_BLU10_BLU10_BLU10_BLU10_BLU10_BLU10_BLU10_BLU10_ILU34_U_ci_large_1
- removed joint BLM1_BLU10_BLU10_BLU10_BLU10_BLU10_BLU10_BLU10_BLU10_BLU10_BLU10_BLU10_BLU10_BLU10_BLU10_BLU10_BLU10_BLU10_BLU10_ILU34_U_ci_large_2
- removed joint BLM1_BLU10_BLU10_BLU10_BLU10_BLU10_BLU10_BLU10_BLU10_BLU10_BLU10_BLU10_BLU10_BLU10_BLU10_BLU10_BLU10_BLU10_JTLU19_U_tj_large_1
- removed joint BLM1_BLU10_BLU10_BLU10_BLU10_BLU10_BLU10_BLU10_BLU10_BLU10_BLU10_BLU10_BLU10_BLU10_BLU10_BLU10_BLU10_BLU10_JTLU19_U_tj_large_2
- removed joint BLM1_BLU10_BLU10_BLU10_BLU10_BLU10_BLU10_BLU10_BLU10_BLU10_BLU10_BLU10_BLU10_BLU10_BLU10_BLU10_BLU10_ILU35_U_ci_large_1
- removed joint BLM1_BLU10_BLU10_BLU10_BLU10_BLU10_BLU10_BLU10_BLU10_BLU10_BLU10_BLU10_BLU10_BLU10_BLU10_BLU10_BLU10_ILU35_U_ci_large_2
- removed joint BLM1_BLU10_BLU10_BLU10_BLU10_BLU10_BLU10_BLU10_BLU10_BLU10_BLU10_BLU10_BLU10_BLU10_BLU10_BLU10_SLMU8_U_sl_large
- removed joint BLM1_BLU10_BLU10_BLU10_BLU10_BLU10_BLU10_BLU10_BLU10_BLU10_BLU10_BLU10_BLU10_BLU10_BLU10_BLU10_SLMU8_U_sl_medium
- removed joint BLM1_BLU10_BLU10_BLU10_BLU10_BLU10_BLU10_BLU10_BLU10_BLU10_BLU10_BLU10_BLU10_BLU10_BLU10_IMU26_U_reverse_U_ic_medium_1
- removed joint BLM1_BLU10_BLU10_BLU10_BLU10_BLU10_BLU10_BLU10_BLU10_BLU10_BLU10_BLU10_BLU10_BLU10_BLU10_IMU26_U_reverse_U_ic_medium_2
- removed joint BLM1_BLU10_BLU10_BLU10_BLU10_BLU10_BLU10_BLU10_BLU10_BLU10_BLU10_BLU10_BLU10_BLU10_JTMU9_U_reverse_U_tj_medium_1
- removed joint BLM1_BLU10_BLU10_BLU10_BLU10_BLU10_BLU10_BLU10_BLU10_BLU10_BLU10_BLU10_BLU10_BLU10_JTMU9_U_reverse_U_tj_medium_2
- removed joint BLM1_BLU10_BLU10_BLU10_BLU10_BLU10_BLU10_BLU10_BLU10_BLU10_BLU10_BLU10_BLU10_IMU27_reverse_IMU27_U_ic_medium_1
- removed joint BLM1_BLU10_BLU10_BLU10_BLU10_BLU10_BLU10_BLU10_BLU10_BLU10_BLU10_BLU10_BLU10_IMU27_reverse_IMU27_U_ic_medium_2
- removed joint BLM1_BLU10_BLU10_BLU10_BLU10_BLU10_BLU10_BLU10_BLU10_BLU10_BLU10_BLU10_CMMU6_U_cl_medium_1
- removed joint BLM1_BLU10_BLU10_BLU10_BLU10_BLU10_BLU10_BLU10_BLU10_BLU10_BLU10_BLU10_CMMU6_U_cl_medium_2
- removed joint BLM1_BLU10_BLU10_BLU10_BLU10_BLU10_BLU10_BLU10_BLU10_BLU10_BLU10_IMU28_U_ic_medium_1
- removed joint BLM1_BLU10_BLU10_BLU10_BLU10_BLU10_BLU10_BLU10_BLU10_BLU10_BLU10_IMU28_U_ic_medium_2
- removed joint BLM1_BLU10_BLU10_BLU10_BLU10_BLU10_BLU10_BLU10_BLU10_BLU10_SMSU5_U_sl_medium
- removed joint BLM1_BLU10_BLU10_BLU10_BLU10_BLU10_BLU10_BLU10_BLU10_BLU10_SMSU5_U_sl_small
- removed joint BLM1_BLU10_BLU10_BLU10_BLU10_BLU10_BLU10_BLU10_BLU10_ISU15_U_reverse_U_ic_small_1
- removed joint BLM1_BLU10_BLU10_BLU10_BLU10_BLU10_BLU10_BLU10_BLU10_ISU15_U_reverse_U_ic_small_2
- removed joint BLM1_BLU10_BLU10_BLU10_BLU10_BLU10_BLU10_BLU10_JSU13_U_reverse_U_tj_small_1
- removed joint BLM1_BLU10_BLU10_BLU10_BLU10_BLU10_BLU10_BLU10_JSU13_U_reverse_U_tj_small_2
- removed joint BLM1_BLU10_BLU10_BLU10_BLU10_BLU10_BLU10_ISU16_U_reverse_U_ic_small_1
- removed joint BLM1_BLU10_BLU10_BLU10_BLU10_BLU10_BLU10_ISU16_U_reverse_U_ic_small_2
- removed joint BLM1_BLU10_BLU10_BLU10_BLU10_BLU10_JSU14_U_reverse_U_tj_small_1
- removed joint BLM1_BLU10_BLU10_BLU10_BLU10_BLU10_JSU14_U_reverse_U_tj_small_2
- removed joint BLM1_BLU10_BLU10_BLU10_BLU10_ISU17_U_reverse_U_ic_small_1
- removed joint BLM1_BLU10_BLU10_BLU10_BLU10_ISU17_U_reverse_U_ic_small_2
- removed joint BLM1_BLU10_BLU10_BLU10_JSU15_U_reverse_U_tj_small_1
- removed joint BLM1_BLU10_BLU10_BLU10_JSU15_U_reverse_U_tj_small_2
- removed joint BLM1_BLU10_BLU10_ISU18_reverse_ISU18_U_ic_small_1
- removed joint BLM1_BLU10_BLU10_ISU18_reverse_ISU18_U_ic_small_2
- removed joint BLM1_BLU10_ESU1_U_e_small
- added joint BLM1_BLU65_BLU65_BLU65_BLU65_BLU65_BLU65_BLU65_BLU65_BLU65_BLU65_BLU65_BLU65_BLU65_BLU65_BLU65_BLU65_BLU65_BLU65_BLU65_BLU65_BLU65_U_b_large: type fixed, parent BLM1_BLU65_BLU65_BLU65_BLU65_BLU65_BLU65_BLU65_BLU65_BLU65_BLU65_BLU65_BLU65_BLU65_BLU65_BLU65_BLU65_BLU65_BLU65_BLU65_BLU65_BLU65_U_b_body, child BLM1_BLU65_BLU65_BLU65_BLU65_BLU65_BLU65_BLU65_BLU65_BLU65_BLU65_BLU65_BLU65_BLU65_BLU65_BLU65_BLU65_BLU65_BLU65_BLU65_BLU65_BLU65_U_b_in, origin xyz=0 0 0.0513 rpy=3.14159265358979 0 0, axis 0 0 1
- added joint BLM1_BLU65_BLU65_BLU65_BLU65_BLU65_BLU65_BLU65_BLU65_BLU65_BLU65_BLU65_BLU65_BLU65_BLU65_BLU65_BLU65_BLU65_BLU65_BLU65_BLU65_ILU188_U_ci_large_1: type fixed, parent BLM1_BLU65_BLU65_BLU65_BLU65_BLU65_BLU65_BLU65_BLU65_BLU65_BLU65_BLU65_BLU65_BLU65_BLU65_BLU65_BLU65_BLU65_BLU65_BLU65_BLU65_BLU65_U_b_in, child BLM1_BLU65_BLU65_BLU65_BLU65_BLU65_BLU65_BLU65_BLU65_BLU65_BLU65_BLU65_BLU65_BLU65_BLU65_BLU65_BLU65_BLU65_BLU65_BLU65_BLU65_ILU188_U_ci_body, origin xyz=0 0 0 rpy=0 0 0, axis 0 0 0
- added joint BLM1_BLU65_BLU65_BLU65_BLU65_BLU65_BLU65_BLU65_BLU65_BLU65_BLU65_BLU65_BLU65_BLU65_BLU65_BLU65_BLU65_BLU65_BLU65_BLU65_BLU65_ILU188_U_ci_large_2: type fixed, parent BLM1_BLU65_BLU65_BLU65_BLU65_BLU65_BLU65_BLU65_BLU65_BLU65_BLU65_BLU65_BLU65_BLU65_BLU65_BLU65_BLU65_BLU65_BLU65_BLU65_BLU65_ILU188_U_ci_body, child BLM1_BLU65_BLU65_BLU65_BLU65_BLU65_BLU65_BLU65_BLU65_BLU65_BLU65_BLU65_BLU65_BLU65_BLU65_BLU65_BLU65_BLU65_BLU65_BLU65_BLU65_ILU188_U_ci_in, origin xyz=0 0 -0.0114 rpy=0 0 0, axis 0 0 0
- added joint BLM1_BLU65_BLU65_BLU65_BLU65_BLU65_BLU65_BLU65_BLU65_BLU65_BLU65_BLU65_BLU65_BLU65_BLU65_BLU65_BLU65_BLU65_BLU65_BLU65_JTLU118_U_tj_large_1: type revolute, parent BLM1_BLU65_BLU65_BLU65_BLU65_BLU65_BLU65_BLU65_BLU65_BLU65_BLU65_BLU65_BLU65_BLU65_BLU65_BLU65_BLU65_BLU65_BLU65_BLU65_BLU65_ILU188_U_ci_in, child BLM1_BLU65_BLU65_BLU65_BLU65_BLU65_BLU65_BLU65_BLU65_BLU65_BLU65_BLU65_BLU65_BLU65_BLU65_BLU65_BLU65_BLU65_BLU65_BLU65_JTLU118_U_tj_body, origin xyz=0.0 0.0 0.0 rpy=0.0 0.0 3.141592653589793, axis 0 0 1, limit lower=-3.1416 upper=3.1416 effort=60.5 velocity=0.33
- added joint BLM1_BLU65_BLU65_BLU65_BLU65_BLU65_BLU65_BLU65_BLU65_BLU65_BLU65_BLU65_BLU65_BLU65_BLU65_BLU65_BLU65_BLU65_BLU65_BLU65_JTLU118_U_tj_large_2: type fixed, parent BLM1_BLU65_BLU65_BLU65_BLU65_BLU65_BLU65_BLU65_BLU65_BLU65_BLU65_BLU65_BLU65_BLU65_BLU65_BLU65_BLU65_BLU65_BLU65_BLU65_JTLU118_U_tj_body, child BLM1_BLU65_BLU65_BLU65_BLU65_BLU65_BLU65_BLU65_BLU65_BLU65_BLU65_BLU65_BLU65_BLU65_BLU65_BLU65_BLU65_BLU65_BLU65_BLU65_JTLU118_U_tj_in, origin xyz=-0.057 0 -0.0735 rpy=0 1.5707963267949 0, axis 0 0 0
- added joint BLM1_BLU65_BLU65_BLU65_BLU65_BLU65_BLU65_BLU65_BLU65_BLU65_BLU65_BLU65_BLU65_BLU65_BLU65_BLU65_BLU65_BLU65_BLU65_ILU189_U_ci_large_1: type fixed, parent BLM1_BLU65_BLU65_BLU65_BLU65_BLU65_BLU65_BLU65_BLU65_BLU65_BLU65_BLU65_BLU65_BLU65_BLU65_BLU65_BLU65_BLU65_BLU65_BLU65_JTLU118_U_tj_in, child BLM1_BLU65_BLU65_BLU65_BLU65_BLU65_BLU65_BLU65_BLU65_BLU65_BLU65_BLU65_BLU65_BLU65_BLU65_BLU65_BLU65_BLU65_BLU65_ILU189_U_ci_body, origin xyz=0 0 0 rpy=0 0 0, axis 0 0 0
- added joint BLM1_BLU65_BLU65_BLU65_BLU65_BLU65_BLU65_BLU65_BLU65_BLU65_BLU65_BLU65_BLU65_BLU65_BLU65_BLU65_BLU65_BLU65_BLU65_ILU189_U_ci_large_2: type fixed, parent BLM1_BLU65_BLU65_BLU65_BLU65_BLU65_BLU65_BLU65_BLU65_BLU65_BLU65_BLU65_BLU65_BLU65_BLU65_BLU65_BLU65_BLU65_BLU65_ILU189_U_ci_body, child BLM1_BLU65_BLU65_BLU65_BLU65_BLU65_BLU65_BLU65_BLU65_BLU65_BLU65_BLU65_BLU65_BLU65_BLU65_BLU65_BLU65_BLU65_BLU65_ILU189_U_ci_in, origin xyz=0 0 -0.0114 rpy=0 0 0, axis 0 0 0
- added joint BLM1_BLU65_BLU65_BLU65_BLU65_BLU65_BLU65_BLU65_BLU65_BLU65_BLU65_BLU65_BLU65_BLU65_BLU65_BLU65_BLU65_BLU65_JTLU119_U_tj_large_1: type revolute, parent BLM1_BLU65_BLU65_BLU65_BLU65_BLU65_BLU65_BLU65_BLU65_BLU65_BLU65_BLU65_BLU65_BLU65_BLU65_BLU65_BLU65_BLU65_BLU65_ILU189_U_ci_in, child BLM1_BLU65_BLU65_BLU65_BLU65_BLU65_BLU65_BLU65_BLU65_BLU65_BLU65_BLU65_BLU65_BLU65_BLU65_BLU65_BLU65_BLU65_JTLU119_U_tj_body, origin xyz=0.0 0.0 0.0 rpy=0.0 0.0 3.141592653589793, axis 0 0 1, limit lower=-3.1416 upper=3.1416 effort=60.5 velocity=0.33
- added joint BLM1_BLU65_BLU65_BLU65_BLU65_BLU65_BLU65_BLU65_BLU65_BLU65_BLU65_BLU65_BLU65_BLU65_BLU65_BLU65_BLU65_BLU65_JTLU119_U_tj_large_2: type fixed, parent BLM1_BLU65_BLU65_BLU65_BLU65_BLU65_BLU65_BLU65_BLU65_BLU65_BLU65_BLU65_BLU65_BLU65_BLU65_BLU65_BLU65_BLU65_JTLU119_U_tj_body, child BLM1_BLU65_BLU65_BLU65_BLU65_BLU65_BLU65_BLU65_BLU65_BLU65_BLU65_BLU65_BLU65_BLU65_BLU65_BLU65_BLU65_BLU65_JTLU119_U_tj_in, origin xyz=-0.057 0 -0.0735 rpy=0 1.5707963267949 0, axis 0 0 0
- added joint BLM1_BLU65_BLU65_BLU65_BLU65_BLU65_BLU65_BLU65_BLU65_BLU65_BLU65_BLU65_BLU65_BLU65_BLU65_BLU65_BLU65_ILU190_U_ci_large_1: type fixed, parent BLM1_BLU65_BLU65_BLU65_BLU65_BLU65_BLU65_BLU65_BLU65_BLU65_BLU65_BLU65_BLU65_BLU65_BLU65_BLU65_BLU65_BLU65_JTLU119_U_tj_in, child BLM1_BLU65_BLU65_BLU65_BLU65_BLU65_BLU65_BLU65_BLU65_BLU65_BLU65_BLU65_BLU65_BLU65_BLU65_BLU65_BLU65_ILU190_U_ci_body, origin xyz=0 0 0 rpy=0 0 0, axis 0 0 0
- added joint BLM1_BLU65_BLU65_BLU65_BLU65_BLU65_BLU65_BLU65_BLU65_BLU65_BLU65_BLU65_BLU65_BLU65_BLU65_BLU65_BLU65_ILU190_U_ci_large_2: type fixed, parent BLM1_BLU65_BLU65_BLU65_BLU65_BLU65_BLU65_BLU65_BLU65_BLU65_BLU65_BLU65_BLU65_BLU65_BLU65_BLU65_BLU65_ILU190_U_ci_body, child BLM1_BLU65_BLU65_BLU65_BLU65_BLU65_BLU65_BLU65_BLU65_BLU65_BLU65_BLU65_BLU65_BLU65_BLU65_BLU65_BLU65_ILU190_U_ci_in, origin xyz=0 0 -0.0114 rpy=0 0 0, axis 0 0 0
- added joint BLM1_BLU65_BLU65_BLU65_BLU65_BLU65_BLU65_BLU65_BLU65_BLU65_BLU65_BLU65_BLU65_BLU65_BLU65_BLU65_SLMU44_U_sl_large: type fixed, parent BLM1_BLU65_BLU65_BLU65_BLU65_BLU65_BLU65_BLU65_BLU65_BLU65_BLU65_BLU65_BLU65_BLU65_BLU65_BLU65_BLU65_ILU190_U_ci_in, child BLM1_BLU65_BLU65_BLU65_BLU65_BLU65_BLU65_BLU65_BLU65_BLU65_BLU65_BLU65_BLU65_BLU65_BLU65_BLU65_SLMU44_U_sl_body, origin xyz=0.0 0.0 0.0 rpy=0.0 0.0 3.141592653589793, axis 0 0 0
- added joint BLM1_BLU65_BLU65_BLU65_BLU65_BLU65_BLU65_BLU65_BLU65_BLU65_BLU65_BLU65_BLU65_BLU65_BLU65_BLU65_SLMU44_U_sl_medium: type fixed, parent BLM1_BLU65_BLU65_BLU65_BLU65_BLU65_BLU65_BLU65_BLU65_BLU65_BLU65_BLU65_BLU65_BLU65_BLU65_BLU65_SLMU44_U_sl_body, child BLM1_BLU65_BLU65_BLU65_BLU65_BLU65_BLU65_BLU65_BLU65_BLU65_BLU65_BLU65_BLU65_BLU65_BLU65_IMU96_U_reverse_U_ic_in, origin xyz=0 0 -0.2 rpy=3.14159265358979 0 0, axis 0 0 0
- added joint BLM1_BLU65_BLU65_BLU65_BLU65_BLU65_BLU65_BLU65_BLU65_BLU65_BLU65_BLU65_BLU65_BLU65_BLU65_IMU96_U_reverse_U_ic_medium_1: type fixed, parent BLM1_BLU65_BLU65_BLU65_BLU65_BLU65_BLU65_BLU65_BLU65_BLU65_BLU65_BLU65_BLU65_BLU65_BLU65_IMU96_U_reverse_U_ic_body, child BLM1_BLU65_BLU65_BLU65_BLU65_BLU65_BLU65_BLU65_BLU65_BLU65_BLU65_BLU65_BLU65_BLU65_JTMU37_U_reverse_U_tj_in, origin xyz=-0.0 -0.0 -0.0 rpy=0.0 0.0 0.0, axis 0 0 0
- added joint BLM1_BLU65_BLU65_BLU65_BLU65_BLU65_BLU65_BLU65_BLU65_BLU65_BLU65_BLU65_BLU65_BLU65_BLU65_IMU96_U_reverse_U_ic_medium_2: type fixed, parent BLM1_BLU65_BLU65_BLU65_BLU65_BLU65_BLU65_BLU65_BLU65_BLU65_BLU65_BLU65_BLU65_BLU65_BLU65_IMU96_U_reverse_U_ic_in, child BLM1_BLU65_BLU65_BLU65_BLU65_BLU65_BLU65_BLU65_BLU65_BLU65_BLU65_BLU65_BLU65_BLU65_BLU65_IMU96_U_reverse_U_ic_body, origin xyz=0.0 0.0 0.0094 rpy=0.0 0.0 3.141592653589793, axis 0 0 0
- added joint BLM1_BLU65_BLU65_BLU65_BLU65_BLU65_BLU65_BLU65_BLU65_BLU65_BLU65_BLU65_BLU65_BLU65_JTMU37_U_reverse_U_tj_medium_1: type revolute, parent BLM1_BLU65_BLU65_BLU65_BLU65_BLU65_BLU65_BLU65_BLU65_BLU65_BLU65_BLU65_BLU65_BLU65_JTMU37_U_reverse_U_tj_body, child BLM1_BLU65_BLU65_BLU65_BLU65_BLU65_BLU65_BLU65_BLU65_BLU65_BLU65_BLU65_BLU65_IMU97_reverse_IMU97_U_ic_in, origin xyz=-0.0 -0.0 -0.0 rpy=0.0 0.0 0.0, axis 0 0 1, limit lower=-3.1416 upper=3.1416 effort=25.5 velocity=0.33
- added joint BLM1_BLU65_BLU65_BLU65_BLU65_BLU65_BLU65_BLU65_BLU65_BLU65_BLU65_BLU65_BLU65_BLU65_JTMU37_U_reverse_U_tj_medium_2: type fixed, parent BLM1_BLU65_BLU65_BLU65_BLU65_BLU65_BLU65_BLU65_BLU65_BLU65_BLU65_BLU65_BLU65_BLU65_JTMU37_U_reverse_U_tj_in, child BLM1_BLU65_BLU65_BLU65_BLU65_BLU65_BLU65_BLU65_BLU65_BLU65_BLU65_BLU65_BLU65_BLU65_JTMU37_U_reverse_U_tj_body, origin xyz=-0.06350000000000017 -0.0 0.04699999999999977 rpy=0.0 -1.5707963267949 0.0, axis 0 -1 0
- added joint BLM1_BLU65_BLU65_BLU65_BLU65_BLU65_BLU65_BLU65_BLU65_BLU65_BLU65_BLU65_BLU65_IMU97_reverse_IMU97_U_ic_medium_1: type fixed, parent BLM1_BLU65_BLU65_BLU65_BLU65_BLU65_BLU65_BLU65_BLU65_BLU65_BLU65_BLU65_BLU65_IMU97_reverse_IMU97_U_ic_body, child BLM1_BLU65_BLU65_BLU65_BLU65_BLU65_BLU65_BLU65_BLU65_BLU65_BLU65_BLU65_CMMU27_U_cl_in_1, origin xyz=-0.0 -0.0 -0.0 rpy=0.0 0.0 3.141592653589793, axis 0 0 0
- added joint BLM1_BLU65_BLU65_BLU65_BLU65_BLU65_BLU65_BLU65_BLU65_BLU65_BLU65_BLU65_BLU65_IMU97_reverse_IMU97_U_ic_medium_2: type fixed, parent BLM1_BLU65_BLU65_BLU65_BLU65_BLU65_BLU65_BLU65_BLU65_BLU65_BLU65_BLU65_BLU65_IMU97_reverse_IMU97_U_ic_in, child BLM1_BLU65_BLU65_BLU65_BLU65_BLU65_BLU65_BLU65_BLU65_BLU65_BLU65_BLU65_BLU65_IMU97_reverse_IMU97_U_ic_body, origin xyz=-0.0 -0.0 0.0094 rpy=0.0 0.0 0.0, axis 0 0 0
- added joint BLM1_BLU65_BLU65_BLU65_BLU65_BLU65_BLU65_BLU65_BLU65_BLU65_BLU65_BLU65_CMMU27_U_cl_medium_1: type fixed, parent BLM1_BLU65_BLU65_BLU65_BLU65_BLU65_BLU65_BLU65_BLU65_BLU65_BLU65_BLU65_CMMU27_U_cl_in_1, child BLM1_BLU65_BLU65_BLU65_BLU65_BLU65_BLU65_BLU65_BLU65_BLU65_BLU65_BLU65_CMMU27_U_cl_body, origin xyz=0 0 0 rpy=0 0 0, axis 0 0 0
- added joint BLM1_BLU65_BLU65_BLU65_BLU65_BLU65_BLU65_BLU65_BLU65_BLU65_BLU65_BLU65_CMMU27_U_cl_medium_2: type fixed, parent BLM1_BLU65_BLU65_BLU65_BLU65_BLU65_BLU65_BLU65_BLU65_BLU65_BLU65_BLU65_CMMU27_U_cl_body, child BLM1_BLU65_BLU65_BLU65_BLU65_BLU65_BLU65_BLU65_BLU65_BLU65_BLU65_BLU65_CMMU27_U_cl_in_2, origin xyz=-0.0635 0 0.047 rpy=0 1.5707963267949 0, axis 0 0 0
- added joint BLM1_BLU65_BLU65_BLU65_BLU65_BLU65_BLU65_BLU65_BLU65_BLU65_BLU65_IMU98_U_ic_medium_1: type fixed, parent BLM1_BLU65_BLU65_BLU65_BLU65_BLU65_BLU65_BLU65_BLU65_BLU65_BLU65_BLU65_CMMU27_U_cl_in_2, child BLM1_BLU65_BLU65_BLU65_BLU65_BLU65_BLU65_BLU65_BLU65_BLU65_BLU65_IMU98_U_ic_body, origin xyz=0 0 0 rpy=0 0 0, axis 0 0 0
- added joint BLM1_BLU65_BLU65_BLU65_BLU65_BLU65_BLU65_BLU65_BLU65_BLU65_BLU65_IMU98_U_ic_medium_2: type fixed, parent BLM1_BLU65_BLU65_BLU65_BLU65_BLU65_BLU65_BLU65_BLU65_BLU65_BLU65_IMU98_U_ic_body, child BLM1_BLU65_BLU65_BLU65_BLU65_BLU65_BLU65_BLU65_BLU65_BLU65_BLU65_IMU98_U_ic_in, origin xyz=0 0 -0.0094 rpy=0 0 0, axis 0 0 0
- added joint BLM1_BLU65_BLU65_BLU65_BLU65_BLU65_BLU65_BLU65_BLU65_BLU65_SMSU20_U_sl_medium: type fixed, parent BLM1_BLU65_BLU65_BLU65_BLU65_BLU65_BLU65_BLU65_BLU65_BLU65_BLU65_IMU98_U_ic_in, child BLM1_BLU65_BLU65_BLU65_BLU65_BLU65_BLU65_BLU65_BLU65_BLU65_SMSU20_U_sl_body, origin xyz=0 0 0 rpy=0 0 0, axis 0 0 0
- added joint BLM1_BLU65_BLU65_BLU65_BLU65_BLU65_BLU65_BLU65_BLU65_BLU65_SMSU20_U_sl_small: type fixed, parent BLM1_BLU65_BLU65_BLU65_BLU65_BLU65_BLU65_BLU65_BLU65_BLU65_SMSU20_U_sl_body, child BLM1_BLU65_BLU65_BLU65_BLU65_BLU65_BLU65_BLU65_BLU65_ISU35_U_reverse_U_ic_in, origin xyz=0 0 -0.2 rpy=3.1416 0 0, axis 0 0 0
- added joint BLM1_BLU65_BLU65_BLU65_BLU65_BLU65_BLU65_BLU65_BLU65_ISU35_U_reverse_U_ic_small_1: type fixed, parent BLM1_BLU65_BLU65_BLU65_BLU65_BLU65_BLU65_BLU65_BLU65_ISU35_U_reverse_U_ic_body, child BLM1_BLU65_BLU65_BLU65_BLU65_BLU65_BLU65_BLU65_JSU32_U_reverse_U_tj_in, origin xyz=-0.0 -0.0 -0.0 rpy=0.0 0.0 0.0, axis 0 0 0
- added joint BLM1_BLU65_BLU65_BLU65_BLU65_BLU65_BLU65_BLU65_BLU65_ISU35_U_reverse_U_ic_small_2: type fixed, parent BLM1_BLU65_BLU65_BLU65_BLU65_BLU65_BLU65_BLU65_BLU65_ISU35_U_reverse_U_ic_in, child BLM1_BLU65_BLU65_BLU65_BLU65_BLU65_BLU65_BLU65_BLU65_ISU35_U_reverse_U_ic_body, origin xyz=0.0 0.0 0.0073 rpy=0.0 0.0 3.141592653589793, axis 0 0 0
- added joint BLM1_BLU65_BLU65_BLU65_BLU65_BLU65_BLU65_BLU65_JSU32_U_reverse_U_tj_small_1: type revolute, parent BLM1_BLU65_BLU65_BLU65_BLU65_BLU65_BLU65_BLU65_JSU32_U_reverse_U_tj_body, child BLM1_BLU65_BLU65_BLU65_BLU65_BLU65_BLU65_ISU36_U_reverse_U_ic_in, origin xyz=-0.0 -0.0 -0.0 rpy=0.0 0.0 0.0, axis 0 0 1, limit lower=-3.1416 upper=3.1416 effort=4.5 velocity=0.4
- added joint BLM1_BLU65_BLU65_BLU65_BLU65_BLU65_BLU65_BLU65_JSU32_U_reverse_U_tj_small_2: type fixed, parent BLM1_BLU65_BLU65_BLU65_BLU65_BLU65_BLU65_BLU65_JSU32_U_reverse_U_tj_in, child BLM1_BLU65_BLU65_BLU65_BLU65_BLU65_BLU65_BLU65_JSU32_U_reverse_U_tj_body, origin xyz=-0.057500000000000134 -0.0 0.036499999999999796 rpy=0.0 -1.5707963267949 0.0, axis 0 0 0
- added joint BLM1_BLU65_BLU65_BLU65_BLU65_BLU65_BLU65_ISU36_U_reverse_U_ic_small_1: type fixed, parent BLM1_BLU65_BLU65_BLU65_BLU65_BLU65_BLU65_ISU36_U_reverse_U_ic_body, child BLM1_BLU65_BLU65_BLU65_BLU65_BLU65_JSU33_U_reverse_U_tj_in, origin xyz=-0.0 -0.0 -0.0 rpy=0.0 0.0 0.0, axis 0 0 0
- added joint BLM1_BLU65_BLU65_BLU65_BLU65_BLU65_BLU65_ISU36_U_reverse_U_ic_small_2: type fixed, parent BLM1_BLU65_BLU65_BLU65_BLU65_BLU65_BLU65_ISU36_U_reverse_U_ic_in, child BLM1_BLU65_BLU65_BLU65_BLU65_BLU65_BLU65_ISU36_U_reverse_U_ic_body, origin xyz=0.0 0.0 0.0073 rpy=0.0 0.0 3.141592653589793, axis 0 0 0
- added joint BLM1_BLU65_BLU65_BLU65_BLU65_BLU65_JSU33_U_reverse_U_tj_small_1: type revolute, parent BLM1_BLU65_BLU65_BLU65_BLU65_BLU65_JSU33_U_reverse_U_tj_body, child BLM1_BLU65_BLU65_BLU65_BLU65_ISU37_U_reverse_U_ic_in, origin xyz=-0.0 -0.0 -0.0 rpy=0.0 0.0 0.0, axis 0 0 1, limit lower=-3.1416 upper=3.1416 effort=4.5 velocity=0.4
- added joint BLM1_BLU65_BLU65_BLU65_BLU65_BLU65_JSU33_U_reverse_U_tj_small_2: type fixed, parent BLM1_BLU65_BLU65_BLU65_BLU65_BLU65_JSU33_U_reverse_U_tj_in, child BLM1_BLU65_BLU65_BLU65_BLU65_BLU65_JSU33_U_reverse_U_tj_body, origin xyz=-0.057500000000000134 -0.0 0.036499999999999796 rpy=0.0 -1.5707963267949 0.0, axis 0 0 0
- added joint BLM1_BLU65_BLU65_BLU65_BLU65_ISU37_U_reverse_U_ic_small_1: type fixed, parent BLM1_BLU65_BLU65_BLU65_BLU65_ISU37_U_reverse_U_ic_body, child BLM1_BLU65_BLU65_BLU65_JSU34_U_reverse_U_tj_in, origin xyz=-0.0 -0.0 -0.0 rpy=0.0 0.0 0.0, axis 0 0 0
- added joint BLM1_BLU65_BLU65_BLU65_BLU65_ISU37_U_reverse_U_ic_small_2: type fixed, parent BLM1_BLU65_BLU65_BLU65_BLU65_ISU37_U_reverse_U_ic_in, child BLM1_BLU65_BLU65_BLU65_BLU65_ISU37_U_reverse_U_ic_body, origin xyz=0.0 0.0 0.0073 rpy=0.0 0.0 3.141592653589793, axis 0 0 0
- added joint BLM1_BLU65_BLU65_BLU65_JSU34_U_reverse_U_tj_small_1: type revolute, parent BLM1_BLU65_BLU65_BLU65_JSU34_U_reverse_U_tj_body, child BLM1_BLU65_BLU65_ISU38_reverse_ISU38_U_ic_in, origin xyz=-0.0 -0.0 -0.0 rpy=0.0 0.0 0.0, axis 0 0 1, limit lower=-3.1416 upper=3.1416 effort=4.5 velocity=0.4
- added joint BLM1_BLU65_BLU65_BLU65_JSU34_U_reverse_U_tj_small_2: type fixed, parent BLM1_BLU65_BLU65_BLU65_JSU34_U_reverse_U_tj_in, child BLM1_BLU65_BLU65_BLU65_JSU34_U_reverse_U_tj_body, origin xyz=-0.057500000000000134 -0.0 0.036499999999999796 rpy=0.0 -1.5707963267949 0.0, axis 0 0 0
- added joint BLM1_BLU65_BLU65_ISU38_reverse_ISU38_U_ic_small_1: type fixed, parent BLM1_BLU65_BLU65_ISU38_reverse_ISU38_U_ic_body, child BLM1_BLU65_ESU2_U_ee_in, origin xyz=-0.0 -0.0 -0.0 rpy=0.0 0.0 0.0, axis 0 0 0
- added joint BLM1_BLU65_BLU65_ISU38_reverse_ISU38_U_ic_small_2: type fixed, parent BLM1_BLU65_BLU65_ISU38_reverse_ISU38_U_ic_in, child BLM1_BLU65_BLU65_ISU38_reverse_ISU38_U_ic_body, origin xyz=-0.0 -0.0 0.0073 rpy=0.0 0.0 0.0, axis 0 0 0
- added joint BLM1_BLU65_ESU2_U_ee_small: type fixed, parent BLM1_BLU65_ESU2_U_ee_in, child BLM1_BLU65_ESU2_U_ee_body, origin xyz=0 0 0 rpy=0 0 0, axis 0 0 0
