Commit message: 🐞 fix(仿真环境): 文件路径
调整为相对路径

File: src/RobotConfigDesignEnv/robotConfigDesign/res/rebot.urdf (robot description, URDF)
Before this commit: robot UNNAMED_78, 3 links, 2 joints
Links:
- removed link SMM5_SMU0_SMU0_U_sl_body
- removed link SMM5_SMU0_SMU0_U_sl_out_1
- removed link SMM5_SMU0_SMU0_U_sl_out_2
- added link EEMM12_IMU6_EMU0_EMU0_U_ee_body, mass 0.0019211; collision mesh filename=package://end_effector_v_m.SLDASM/meshes/ee_body.STL; visual mesh filename=package://end_effector_v_m.SLDASM/meshes/ee_body.STL
- added link EEMM12_IMU6_EMU0_EMU0_U_ee_in, mass 0.0019211; collision mesh filename=package://end_effector_v_m.SLDASM/meshes/ee_in.STL; visual mesh filename=package://end_effector_v_m.SLDASM/meshes/ee_in.STL
- added link EEMM12_IMU6_IMU6_reverse_IMU6_IMU6_U_ic_body, mass 0; collision mesh filename=package://input_connector_m.SLDASM/meshes/ic_body.STL; visual mesh filename=package://input_connector_m.SLDASM/meshes/ic_body.STL
- added link EEMM12_IMU6_IMU6_reverse_IMU6_IMU6_U_ic_in, mass 0.50882; collision mesh filename=package://input_connector_m.SLDASM/meshes/ic_in.STL; visual mesh filename=package://input_connector_m.SLDASM/meshes/ic_in.STL
Joints:
- removed joint SMM5_SMU0_SMU0_U_sl_medium_1
- removed joint SMM5_SMU0_SMU0_U_sl_medium_2
- added joint EEMM12_IMU6_EMU0_EMU0_U_ee_medium: type fixed, parent EEMM12_IMU6_EMU0_EMU0_U_ee_in, child EEMM12_IMU6_EMU0_EMU0_U_ee_body, origin xyz=0 0 0 rpy=0 0 0, axis 0 0 0
- added joint EEMM12_IMU6_IMU6_reverse_IMU6_IMU6_U_ic_medium_1: type fixed, parent EEMM12_IMU6_IMU6_reverse_IMU6_IMU6_U_ic_body, child EEMM12_IMU6_EMU0_EMU0_U_ee_in, origin xyz=-0.0 -0.0 -0.0 rpy=0.0 0.0 0.0, axis 0 0 0
- added joint EEMM12_IMU6_IMU6_reverse_IMU6_IMU6_U_ic_medium_2: type fixed, parent EEMM12_IMU6_IMU6_reverse_IMU6_IMU6_U_ic_in, child EEMM12_IMU6_IMU6_reverse_IMU6_IMU6_U_ic_body, origin xyz=-0.0 -0.0 0.0094 rpy=0.0 0.0 0.0, axis 0 0 0

Commit message: train-1

File: src/RobotConfigDesignEnv/robotConfigDesign/res/rebot.urdf (robot description, URDF)
Before this commit: robot UNNAMED_202, 4 links, 3 joints
Links:
- removed link EEMM12_IMU6_EMU0_EMU0_U_ee_body
- removed link EEMM12_IMU6_EMU0_EMU0_U_ee_in
- removed link EEMM12_IMU6_IMU6_reverse_IMU6_IMU6_U_ic_body
- removed link EEMM12_IMU6_IMU6_reverse_IMU6_IMU6_U_ic_in
- added link EELM32276_ILU5_ELU0_ELU0_U_ee_body, mass 0.05413; collision mesh filename=package://end_effector_v_l.SLDASM/meshes/ee_body.STL; visual mesh filename=package://end_effector_v_l.SLDASM/meshes/ee_body.STL
- added link EELM32276_ILU5_ELU0_ELU0_U_ee_in, mass 0; collision mesh filename=package://end_effector_v_l.SLDASM/meshes/ee_in.STL; visual mesh filename=package://end_effector_v_l.SLDASM/meshes/ee_in.STL
- added link EELM32276_ILU5_ILU5_reverse_ILU5_ILU5_U_ci_body, mass 0; collision mesh filename=package://input_connector_l.SLDASM/meshes/ci_body.STL; visual mesh filename=package://input_connector_l.SLDASM/meshes/ci_body.STL
- added link EELM32276_ILU5_ILU5_reverse_ILU5_ILU5_U_ci_in, mass 0; collision mesh filename=package://input_connector_l.SLDASM/meshes/ci_in.STL; visual mesh filename=package://input_connector_l.SLDASM/meshes/ci_in.STL
Joints:
- removed joint EEMM12_IMU6_EMU0_EMU0_U_ee_medium
- removed joint EEMM12_IMU6_IMU6_reverse_IMU6_IMU6_U_ic_medium_1
- removed joint EEMM12_IMU6_IMU6_reverse_IMU6_IMU6_U_ic_medium_2
- added joint EELM32276_ILU5_ELU0_ELU0_U_ee_large: type fixed, parent EELM32276_ILU5_ELU0_ELU0_U_ee_in, child EELM32276_ILU5_ELU0_ELU0_U_ee_body, origin xyz=0 0 0 rpy=0 0 0, axis 0 0 0
- added joint EELM32276_ILU5_ILU5_reverse_ILU5_ILU5_U_ci_large_1: type fixed, parent EELM32276_ILU5_ILU5_reverse_ILU5_ILU5_U_ci_body, child EELM32276_ILU5_ELU0_ELU0_U_ee_in, origin xyz=-0.0 -0.0 -0.0 rpy=0.0 0.0 0.0, axis 0 0 0
- added joint EELM32276_ILU5_ILU5_reverse_ILU5_ILU5_U_ci_large_2: type fixed, parent EELM32276_ILU5_ILU5_reverse_ILU5_ILU5_U_ci_in, child EELM32276_ILU5_ILU5_reverse_ILU5_ILU5_U_ci_body, origin xyz=-0.0 -0.0 0.0114 rpy=0.0 0.0 0.0, axis 0 0 0

Commit message: ✨ feat(环境): 奖励函数
平衡固定惩罚项，削弱构型惩罚项

File: src/RobotConfigDesignEnv/robotConfigDesign/res/rebot.urdf (robot description, URDF)
Before this commit: robot UNNAMED_202, 4 links, 3 joints
Links:
- removed link EEMM12_IMU6_EMU0_EMU0_U_ee_body
- removed link EEMM12_IMU6_EMU0_EMU0_U_ee_in
- removed link EEMM12_IMU6_IMU6_reverse_IMU6_IMU6_U_ic_body
- removed link EEMM12_IMU6_IMU6_reverse_IMU6_IMU6_U_ic_in
- added link SLM80_SLU0_SLU0_U_sl_body, mass 0.42412; collision mesh filename=package://straight_link-l.SLDASM/meshes/sl_body.STL; visual mesh filename=package://straight_link-l.SLDASM/meshes/sl_body.STL
- added link SLM80_SLU0_SLU0_U_sl_out_1, mass 0.42412; collision mesh filename=package://straight_link-l.SLDASM/meshes/sl_out_1.STL; visual mesh filename=package://straight_link-l.SLDASM/meshes/sl_out_1.STL
- added link SLM80_SLU0_SLU0_U_sl_out_2, mass 0.42412; collision mesh filename=package://straight_link-l.SLDASM/meshes/sl_out_2.STL; visual mesh filename=package://straight_link-l.SLDASM/meshes/sl_out_2.STL
Joints:
- removed joint EEMM12_IMU6_EMU0_EMU0_U_ee_medium
- removed joint EEMM12_IMU6_IMU6_reverse_IMU6_IMU6_U_ic_medium_1
- removed joint EEMM12_IMU6_IMU6_reverse_IMU6_IMU6_U_ic_medium_2
- added joint SLM80_SLU0_SLU0_U_sl_large_1: type fixed, parent SLM80_SLU0_SLU0_U_sl_out_1, child SLM80_SLU0_SLU0_U_sl_body, origin xyz=0 0 0 rpy=0 0 0, axis 0 0 0
- added joint SLM80_SLU0_SLU0_U_sl_large_2: type fixed, parent SLM80_SLU0_SLU0_U_sl_body, child SLM80_SLU0_SLU0_U_sl_out_2, origin xyz=0 0 -0.15 rpy=3.14159265358979 0 0, axis 0 0 0

Commit message: RDS训练-v2

File: src/RobotConfigDesignEnv/robotConfigDesign/res/rebot.urdf (robot description, URDF)
Before this commit: robot UNNAMED_208, 3 links, 2 joints
Links:
- removed link SLM80_SLU0_SLU0_U_sl_body
- removed link SLM80_SLU0_SLU0_U_sl_out_1
- removed link SLM80_SLU0_SLU0_U_sl_out_2
- added link BLM177434_BLU392635_BLU392635_BLU392635_BLU392635_BLU392635_U_b_body, mass 0; collision mesh filename=package://base-l.SLDASM/meshes/b_body.STL; visual mesh filename=package://base-l.SLDASM/meshes/b_body.STL
- added link BLM177434_BLU392635_BLU392635_BLU392635_BLU392635_BLU392635_U_b_in, mass 5.9754; collision mesh filename=package://base-l.SLDASM/meshes/b_in.STL; visual mesh filename=package://base-l.SLDASM/meshes/b_in.STL
- added link BLM177434_BLU392635_BLU392635_BLU392635_BLU392635_ILU436215_U_ci_body, mass 0; collision mesh filename=package://input_connector_l.SLDASM/meshes/ci_body.STL; visual mesh filename=package://input_connector_l.SLDASM/meshes/ci_body.STL
- added link BLM177434_BLU392635_BLU392635_BLU392635_BLU392635_ILU436215_U_ci_in, mass 0; collision mesh filename=package://input_connector_l.SLDASM/meshes/ci_in.STL; visual mesh filename=package://input_connector_l.SLDASM/meshes/ci_in.STL
- added link BLM177434_BLU392635_BLU392635_BLU392635_SLU217527_U_sl_body, mass 0.42412; collision mesh filename=package://straight_link-l.SLDASM/meshes/sl_body.STL; visual mesh filename=package://straight_link-l.SLDASM/meshes/sl_body.STL
- added link BLM177434_BLU392635_BLU392635_ILU436216_U_reverse_U_ci_body, mass 0; collision mesh filename=package://input_connector_l.SLDASM/meshes/ci_body.STL; visual mesh filename=package://input_connector_l.SLDASM/meshes/ci_body.STL
- added link BLM177434_BLU392635_BLU392635_ILU436216_U_reverse_U_ci_in, mass 0; collision mesh filename=package://input_connector_l.SLDASM/meshes/ci_in.STL; visual mesh filename=package://input_connector_l.SLDASM/meshes/ci_in.STL
- added link BLM177434_BLU392635_BLU392636_U_reverse_U_b_body, mass 0; collision mesh filename=package://base-l.SLDASM/meshes/b_body.STL; visual mesh filename=package://base-l.SLDASM/meshes/b_body.STL
- added link BLM177434_BLU392635_BLU392636_U_reverse_U_b_in, mass 5.9754; collision mesh filename=package://base-l.SLDASM/meshes/b_in.STL; visual mesh filename=package://base-l.SLDASM/meshes/b_in.STL
Joints:
- removed joint SLM80_SLU0_SLU0_U_sl_large_1
- removed joint SLM80_SLU0_SLU0_U_sl_large_2
- added joint BLM177434_BLU392635_BLU392635_BLU392635_BLU392635_BLU392635_U_b_large: type fixed, parent BLM177434_BLU392635_BLU392635_BLU392635_BLU392635_BLU392635_U_b_body, child BLM177434_BLU392635_BLU392635_BLU392635_BLU392635_BLU392635_U_b_in, origin xyz=0 0 0.0513 rpy=3.14159265358979 0 0, axis 0 0 1
- added joint BLM177434_BLU392635_BLU392635_BLU392635_BLU392635_ILU436215_U_ci_large_1: type fixed, parent BLM177434_BLU392635_BLU392635_BLU392635_BLU392635_BLU392635_U_b_in, child BLM177434_BLU392635_BLU392635_BLU392635_BLU392635_ILU436215_U_ci_body, origin xyz=0 0 0 rpy=0 0 0, axis 0 0 0
- added joint BLM177434_BLU392635_BLU392635_BLU392635_BLU392635_ILU436215_U_ci_large_2: type fixed, parent BLM177434_BLU392635_BLU392635_BLU392635_BLU392635_ILU436215_U_ci_body, child BLM177434_BLU392635_BLU392635_BLU392635_BLU392635_ILU436215_U_ci_in, origin xyz=0 0 -0.0114 rpy=0 0 0, axis 0 0 0
- added joint BLM177434_BLU392635_BLU392635_BLU392635_SLU217527_U_sl_large_1: type fixed, parent BLM177434_BLU392635_BLU392635_BLU392635_BLU392635_ILU436215_U_ci_in, child BLM177434_BLU392635_BLU392635_BLU392635_SLU217527_U_sl_body, origin xyz=0 0 0 rpy=0 0 0, axis 0 0 0
- added joint BLM177434_BLU392635_BLU392635_BLU392635_SLU217527_U_sl_large_2: type fixed, parent BLM177434_BLU392635_BLU392635_BLU392635_SLU217527_U_sl_body, child BLM177434_BLU392635_BLU392635_ILU436216_U_reverse_U_ci_in, origin xyz=0 0 -0.15 rpy=3.14159265358979 0 0, axis 0 0 0
- added joint BLM177434_BLU392635_BLU392635_ILU436216_U_reverse_U_ci_large_1: type fixed, parent BLM177434_BLU392635_BLU392635_ILU436216_U_reverse_U_ci_body, child BLM177434_BLU392635_BLU392636_U_reverse_U_b_in, origin xyz=-0.0 -0.0 -0.0 rpy=0.0 0.0 0.0, axis 0 0 0
- added joint BLM177434_BLU392635_BLU392635_ILU436216_U_reverse_U_ci_large_2: type fixed, parent BLM177434_BLU392635_BLU392635_ILU436216_U_reverse_U_ci_in, child BLM177434_BLU392635_BLU392635_ILU436216_U_reverse_U_ci_body, origin xyz=-0.0 -0.0 0.0114 rpy=0.0 0.0 0.0, axis 0 0 0
- added joint BLM177434_BLU392635_BLU392636_U_reverse_U_b_large: type fixed, parent BLM177434_BLU392635_BLU392636_U_reverse_U_b_in, child BLM177434_BLU392635_BLU392636_U_reverse_U_b_body, origin xyz=-0.0 -1.6575487333678338e-16 0.0513 rpy=3.141592653589793 0.0 0.0, axis 0 0 1

Commit message: 🐞 fix(RL环境): 奖励函数
鼓励agent添加模块，并且将质量惩罚转移到IK评估处

File: src/RobotConfigDesignEnv/robotConfigDesign/res/rebot.urdf (robot description, URDF)
Before this commit: robot UNNAMED_209509, 9 links, 8 joints
Links:
- removed link BLM177434_BLU392635_BLU392635_BLU392635_BLU392635_BLU392635_U_b_body
- removed link BLM177434_BLU392635_BLU392635_BLU392635_BLU392635_BLU392635_U_b_in
- removed link BLM177434_BLU392635_BLU392635_BLU392635_BLU392635_ILU436215_U_ci_body
- removed link BLM177434_BLU392635_BLU392635_BLU392635_BLU392635_ILU436215_U_ci_in
- removed link BLM177434_BLU392635_BLU392635_BLU392635_SLU217527_U_sl_body
- removed link BLM177434_BLU392635_BLU392635_ILU436216_U_reverse_U_ci_body
- removed link BLM177434_BLU392635_BLU392635_ILU436216_U_reverse_U_ci_in
- removed link BLM177434_BLU392635_BLU392636_U_reverse_U_b_body
- removed link BLM177434_BLU392635_BLU392636_U_reverse_U_b_in
- added link BLM27_BLU0_BLU0_BLU0_U_b_body, mass 0; collision mesh filename=package://base-l.SLDASM/meshes/b_body.STL; visual mesh filename=package://base-l.SLDASM/meshes/b_body.STL
- added link BLM27_BLU0_BLU0_BLU0_U_b_in, mass 5.9754; collision mesh filename=package://base-l.SLDASM/meshes/b_in.STL; visual mesh filename=package://base-l.SLDASM/meshes/b_in.STL
- added link BLM27_BLU0_ILU0_ILU0_U_ci_body, mass 0; collision mesh filename=package://input_connector_l.SLDASM/meshes/ci_body.STL; visual mesh filename=package://input_connector_l.SLDASM/meshes/ci_body.STL
- added link BLM27_BLU0_ILU0_ILU0_U_ci_in, mass 0; collision mesh filename=package://input_connector_l.SLDASM/meshes/ci_in.STL; visual mesh filename=package://input_connector_l.SLDASM/meshes/ci_in.STL
Joints:
- removed joint BLM177434_BLU392635_BLU392635_BLU392635_BLU392635_BLU392635_U_b_large
- removed joint BLM177434_BLU392635_BLU392635_BLU392635_BLU392635_ILU436215_U_ci_large_1
- removed joint BLM177434_BLU392635_BLU392635_BLU392635_BLU392635_ILU436215_U_ci_large_2
- removed joint BLM177434_BLU392635_BLU392635_BLU392635_SLU217527_U_sl_large_1
- removed joint BLM177434_BLU392635_BLU392635_BLU392635_SLU217527_U_sl_large_2
- removed joint BLM177434_BLU392635_BLU392635_ILU436216_U_reverse_U_ci_large_1
- removed joint BLM177434_BLU392635_BLU392635_ILU436216_U_reverse_U_ci_large_2
- removed joint BLM177434_BLU392635_BLU392636_U_reverse_U_b_large
- added joint BLM27_BLU0_BLU0_BLU0_U_b_large: type fixed, parent BLM27_BLU0_BLU0_BLU0_U_b_body, child BLM27_BLU0_BLU0_BLU0_U_b_in, origin xyz=0 0 0.0513 rpy=3.14159265358979 0 0, axis 0 0 1
- added joint BLM27_BLU0_ILU0_ILU0_U_ci_large_1: type fixed, parent BLM27_BLU0_BLU0_BLU0_U_b_in, child BLM27_BLU0_ILU0_ILU0_U_ci_body, origin xyz=0 0 0 rpy=0 0 0, axis 0 0 0
- added joint BLM27_BLU0_ILU0_ILU0_U_ci_large_2: type fixed, parent BLM27_BLU0_ILU0_ILU0_U_ci_body, child BLM27_BLU0_ILU0_ILU0_U_ci_in, origin xyz=0 0 -0.0114 rpy=0 0 0, axis 0 0 0

Commit message: 🐞 fix(URDF 生成): Arrangement类
修复返回构型类型列表为Enum而非int的bug

File: src/RobotConfigDesignEnv/robotConfigDesign/res/rebot.urdf (robot description, URDF)
Before this commit: robot UNNAMED_319, 4 links, 3 joints
Links:
- removed link BLM27_BLU0_BLU0_BLU0_U_b_body
- removed link BLM27_BLU0_BLU0_BLU0_U_b_in
- removed link BLM27_BLU0_ILU0_ILU0_U_ci_body
- removed link BLM27_BLU0_ILU0_ILU0_U_ci_in
- added link EELM31_ILU5_ELU0_ELU0_U_ee_body, mass 0.05413; collision mesh filename=package://end_effector_v_l.SLDASM/meshes/ee_body.STL; visual mesh filename=package://end_effector_v_l.SLDASM/meshes/ee_body.STL
- added link EELM31_ILU5_ELU0_ELU0_U_ee_in, mass 0; collision mesh filename=package://end_effector_v_l.SLDASM/meshes/ee_in.STL; visual mesh filename=package://end_effector_v_l.SLDASM/meshes/ee_in.STL
- added link EELM31_ILU5_ILU5_reverse_ILU5_ILU5_U_ci_body, mass 0; collision mesh filename=package://input_connector_l.SLDASM/meshes/ci_body.STL; visual mesh filename=package://input_connector_l.SLDASM/meshes/ci_body.STL
- added link EELM31_ILU5_ILU5_reverse_ILU5_ILU5_U_ci_in, mass 0; collision mesh filename=package://input_connector_l.SLDASM/meshes/ci_in.STL; visual mesh filename=package://input_connector_l.SLDASM/meshes/ci_in.STL
Joints:
- removed joint BLM27_BLU0_BLU0_BLU0_U_b_large
- removed joint BLM27_BLU0_ILU0_ILU0_U_ci_large_1
- removed joint BLM27_BLU0_ILU0_ILU0_U_ci_large_2
- added joint EELM31_ILU5_ELU0_ELU0_U_ee_large: type fixed, parent EELM31_ILU5_ELU0_ELU0_U_ee_in, child EELM31_ILU5_ELU0_ELU0_U_ee_body, origin xyz=0 0 0 rpy=0 0 0, axis 0 0 0
- added joint EELM31_ILU5_ILU5_reverse_ILU5_ILU5_U_ci_large_1: type fixed, parent EELM31_ILU5_ILU5_reverse_ILU5_ILU5_U_ci_body, child EELM31_ILU5_ELU0_ELU0_U_ee_in, origin xyz=-0.0 -0.0 -0.0 rpy=0.0 0.0 0.0, axis 0 0 0
- added joint EELM31_ILU5_ILU5_reverse_ILU5_ILU5_U_ci_large_2: type fixed, parent EELM31_ILU5_ILU5_reverse_ILU5_ILU5_U_ci_in, child EELM31_ILU5_ILU5_reverse_ILU5_ILU5_U_ci_body, origin xyz=-0.0 -0.0 0.0114 rpy=0.0 0.0 0.0, axis 0 0 0
