Commit message: train-v3

File: src/RobotConfigDesignEnv/robotConfigDesign/res/rebot.urdf (robot description, URDF)
Before this commit: robot UNNAMED_220, 4 links, 3 joints
Links:
- removed link EELM31_ILU5_ELU0_ELU0_U_ee_body
- removed link EELM31_ILU5_ELU0_ELU0_U_ee_in
- removed link EELM31_ILU5_ILU5_reverse_ILU5_ILU5_U_ci_body
- removed link EELM31_ILU5_ILU5_reverse_ILU5_ILU5_U_ci_in
- added link JLM3915_JTLU60926_EMU19485_U_ee_body, mass 0.0019211; collision mesh filename=package://end_effector_v_m.SLDASM/meshes/ee_body.STL; visual mesh filename=package://end_effector_v_m.SLDASM/meshes/ee_body.STL
- added link JLM3915_JTLU60926_EMU19485_U_ee_in, mass 0.0019211; collision mesh filename=package://end_effector_v_m.SLDASM/meshes/ee_in.STL; visual mesh filename=package://end_effector_v_m.SLDASM/meshes/ee_in.STL
- added link JLM3915_JTLU60926_JTLU60926_IMU127903_reverse_IMU127903_U_ic_body, mass 0; collision mesh filename=package://input_connector_m.SLDASM/meshes/ic_body.STL; visual mesh filename=package://input_connector_m.SLDASM/meshes/ic_body.STL
- added link JLM3915_JTLU60926_JTLU60926_IMU127903_reverse_IMU127903_U_ic_in, mass 0.50882; collision mesh filename=package://input_connector_m.SLDASM/meshes/ic_in.STL; visual mesh filename=package://input_connector_m.SLDASM/meshes/ic_in.STL
- added link JLM3915_JTLU60926_JTLU60926_JTLU60926_JTLU60926_ILU174538_U_ci_body, mass 0; collision mesh filename=package://input_connector_l.SLDASM/meshes/ci_body.STL; visual mesh filename=package://input_connector_l.SLDASM/meshes/ci_body.STL
- added link JLM3915_JTLU60926_JTLU60926_JTLU60926_JTLU60926_ILU174538_U_ci_in, mass 0; collision mesh filename=package://input_connector_l.SLDASM/meshes/ci_in.STL; visual mesh filename=package://input_connector_l.SLDASM/meshes/ci_in.STL
- added link JLM3915_JTLU60926_JTLU60926_JTLU60926_JTLU60926_JTLU60926_CLMU68943_U_cl_body, mass 1.5378; collision mesh filename=package://corner_link-lm.SLDASM/meshes/cl_body.STL; visual mesh filename=package://corner_link-lm.SLDASM/meshes/cl_body.STL
- added link JLM3915_JTLU60926_JTLU60926_JTLU60926_JTLU60926_JTLU60926_CLMU68943_U_cl_in_1, mass 1.5378; collision mesh filename=package://corner_link-lm.SLDASM/meshes/cl_in_1.STL; visual mesh filename=package://corner_link-lm.SLDASM/meshes/cl_in_1.STL
- added link JLM3915_JTLU60926_JTLU60926_JTLU60926_JTLU60926_JTLU60926_CLMU68943_U_cl_in_2, mass 1.5378; collision mesh filename=package://corner_link-lm.SLDASM/meshes/cl_in_2.STL; visual mesh filename=package://corner_link-lm.SLDASM/meshes/cl_in_2.STL
- added link JLM3915_JTLU60926_JTLU60926_JTLU60926_JTLU60926_JTLU60926_JTLU60926_IMU127902_reverse_IMU127902_U_ic_body, mass 0; collision mesh filename=package://input_connector_m.SLDASM/meshes/ic_body.STL; visual mesh filename=package://input_connector_m.SLDASM/meshes/ic_body.STL
- added link JLM3915_JTLU60926_JTLU60926_JTLU60926_JTLU60926_JTLU60926_JTLU60926_IMU127902_reverse_IMU127902_U_ic_in, mass 0.50882; collision mesh filename=package://input_connector_m.SLDASM/meshes/ic_in.STL; visual mesh filename=package://input_connector_m.SLDASM/meshes/ic_in.STL
- added link JLM3915_JTLU60926_JTLU60926_JTLU60926_JTLU60926_JTLU60926_JTLU60926_JTLU60926_JTLU60926_ILU174537_U_ci_body, mass 0; collision mesh filename=package://input_connector_l.SLDASM/meshes/ci_body.STL; visual mesh filename=package://input_connector_l.SLDASM/meshes/ci_body.STL
- added link JLM3915_JTLU60926_JTLU60926_JTLU60926_JTLU60926_JTLU60926_JTLU60926_JTLU60926_JTLU60926_ILU174537_U_ci_in, mass 0; collision mesh filename=package://input_connector_l.SLDASM/meshes/ci_in.STL; visual mesh filename=package://input_connector_l.SLDASM/meshes/ci_in.STL
- added link JLM3915_JTLU60926_JTLU60926_JTLU60926_JTLU60926_JTLU60926_JTLU60926_JTLU60926_JTLU60926_JTLU60926_U_tj_body, mass 1.5884; collision mesh filename=package://jointT-l.SLDASM/meshes/tj_body.STL; visual mesh filename=package://jointT-l.SLDASM/meshes/tj_body.STL
- added link JLM3915_JTLU60926_JTLU60926_JTLU60926_JTLU60926_JTLU60926_JTLU60926_JTLU60926_JTLU60926_JTLU60926_U_tj_in, mass 1.5884; collision mesh filename=package://jointT-l.SLDASM/meshes/tj_in.STL; visual mesh filename=package://jointT-l.SLDASM/meshes/tj_in.STL
- added link JLM3915_JTLU60926_JTLU60926_JTLU60926_JTLU60926_JTLU60926_JTLU60926_JTLU60926_JTLU60926_JTLU60926_U_tj_out, mass 1.5884; collision mesh filename=package://jointT-l.SLDASM/meshes/tj_out.STL; visual mesh filename=package://jointT-l.SLDASM/meshes/tj_out.STL
- added link JLM3915_JTLU60926_JTLU60926_JTLU60926_JTLU60926_JTLU60926_JTLU60926_JTLU60926_SLMU125823_U_sl_body, mass 1.4196; collision mesh filename=package://straight_link-lm.SLDASM/meshes/sl_body.STL; visual mesh filename=package://straight_link-lm.SLDASM/meshes/sl_body.STL
- added link JLM3915_JTLU60926_JTLU60926_JTLU60926_SLMU125824_U_sl_body, mass 1.4196; collision mesh filename=package://straight_link-lm.SLDASM/meshes/sl_body.STL; visual mesh filename=package://straight_link-lm.SLDASM/meshes/sl_body.STL
Joints:
- removed joint EELM31_ILU5_ELU0_ELU0_U_ee_large
- removed joint EELM31_ILU5_ILU5_reverse_ILU5_ILU5_U_ci_large_1
- removed joint EELM31_ILU5_ILU5_reverse_ILU5_ILU5_U_ci_large_2
- added joint JLM3915_JTLU60926_EMU19485_U_ee_medium: type fixed, parent JLM3915_JTLU60926_EMU19485_U_ee_in, child JLM3915_JTLU60926_EMU19485_U_ee_body, origin xyz=0 0 0 rpy=0 0 0, axis 0 0 0
- added joint JLM3915_JTLU60926_JTLU60926_IMU127903_reverse_IMU127903_U_ic_medium_1: type fixed, parent JLM3915_JTLU60926_JTLU60926_IMU127903_reverse_IMU127903_U_ic_body, child JLM3915_JTLU60926_EMU19485_U_ee_in, origin xyz=-0.0 -0.0 -0.0 rpy=0.0 0.0 0.0, axis 0 0 0
- added joint JLM3915_JTLU60926_JTLU60926_IMU127903_reverse_IMU127903_U_ic_medium_2: type fixed, parent JLM3915_JTLU60926_JTLU60926_IMU127903_reverse_IMU127903_U_ic_in, child JLM3915_JTLU60926_JTLU60926_IMU127903_reverse_IMU127903_U_ic_body, origin xyz=-0.0 -0.0 0.0094 rpy=0.0 0.0 0.0, axis 0 0 0
- added joint JLM3915_JTLU60926_JTLU60926_JTLU60926_JTLU60926_ILU174538_U_ci_large_1: type fixed, parent JLM3915_JTLU60926_JTLU60926_JTLU60926_JTLU60926_JTLU60926_CLMU68943_U_cl_in_2, child JLM3915_JTLU60926_JTLU60926_JTLU60926_JTLU60926_ILU174538_U_ci_body, origin xyz=0 0 0 rpy=0 0 0, axis 0 0 0
- added joint JLM3915_JTLU60926_JTLU60926_JTLU60926_JTLU60926_ILU174538_U_ci_large_2: type fixed, parent JLM3915_JTLU60926_JTLU60926_JTLU60926_JTLU60926_ILU174538_U_ci_body, child JLM3915_JTLU60926_JTLU60926_JTLU60926_JTLU60926_ILU174538_U_ci_in, origin xyz=0 0 -0.0114 rpy=0 0 0, axis 0 0 0
- added joint JLM3915_JTLU60926_JTLU60926_JTLU60926_JTLU60926_JTLU60926_CLMU68943_U_cl_large: type fixed, parent JLM3915_JTLU60926_JTLU60926_JTLU60926_JTLU60926_JTLU60926_CLMU68943_U_cl_body, child JLM3915_JTLU60926_JTLU60926_JTLU60926_JTLU60926_JTLU60926_CLMU68943_U_cl_in_2, origin xyz=-0.0735 0 0.057 rpy=0 1.5707963267949 0, axis 0 0 0
- added joint JLM3915_JTLU60926_JTLU60926_JTLU60926_JTLU60926_JTLU60926_CLMU68943_U_cl_medium: type fixed, parent JLM3915_JTLU60926_JTLU60926_JTLU60926_JTLU60926_JTLU60926_CLMU68943_U_cl_in_1, child JLM3915_JTLU60926_JTLU60926_JTLU60926_JTLU60926_JTLU60926_CLMU68943_U_cl_body, origin xyz=0 0 0 rpy=0 0 0, axis 0 0 0
- added joint JLM3915_JTLU60926_JTLU60926_JTLU60926_JTLU60926_JTLU60926_JTLU60926_IMU127902_reverse_IMU127902_U_ic_medium_1: type fixed, parent JLM3915_JTLU60926_JTLU60926_JTLU60926_JTLU60926_JTLU60926_JTLU60926_IMU127902_reverse_IMU127902_U_ic_body, child JLM3915_JTLU60926_JTLU60926_JTLU60926_JTLU60926_JTLU60926_CLMU68943_U_cl_in_1, origin xyz=-0.0 -0.0 -0.0 rpy=0.0 0.0 3.141592653589793, axis 0 0 0
- added joint JLM3915_JTLU60926_JTLU60926_JTLU60926_JTLU60926_JTLU60926_JTLU60926_IMU127902_reverse_IMU127902_U_ic_medium_2: type fixed, parent JLM3915_JTLU60926_JTLU60926_JTLU60926_JTLU60926_JTLU60926_JTLU60926_IMU127902_reverse_IMU127902_U_ic_in, child JLM3915_JTLU60926_JTLU60926_JTLU60926_JTLU60926_JTLU60926_JTLU60926_IMU127902_reverse_IMU127902_U_ic_body, origin xyz=-0.0 -0.0 0.0094 rpy=0.0 0.0 0.0, axis 0 0 0
- added joint JLM3915_JTLU60926_JTLU60926_JTLU60926_JTLU60926_JTLU60926_JTLU60926_JTLU60926_JTLU60926_ILU174537_U_ci_large_1: type fixed, parent JLM3915_JTLU60926_JTLU60926_JTLU60926_JTLU60926_JTLU60926_JTLU60926_JTLU60926_JTLU60926_JTLU60926_U_tj_in, child JLM3915_JTLU60926_JTLU60926_JTLU60926_JTLU60926_JTLU60926_JTLU60926_JTLU60926_JTLU60926_ILU174537_U_ci_body, origin xyz=0 0 0 rpy=0 0 0, axis 0 0 0
- added joint JLM3915_JTLU60926_JTLU60926_JTLU60926_JTLU60926_JTLU60926_JTLU60926_JTLU60926_JTLU60926_ILU174537_U_ci_large_2: type fixed, parent JLM3915_JTLU60926_JTLU60926_JTLU60926_JTLU60926_JTLU60926_JTLU60926_JTLU60926_JTLU60926_ILU174537_U_ci_body, child JLM3915_JTLU60926_JTLU60926_JTLU60926_JTLU60926_JTLU60926_JTLU60926_JTLU60926_JTLU60926_ILU174537_U_ci_in, origin xyz=0 0 -0.0114 rpy=0 0 0, axis 0 0 0
- added joint JLM3915_JTLU60926_JTLU60926_JTLU60926_JTLU60926_JTLU60926_JTLU60926_JTLU60926_JTLU60926_JTLU60926_U_tj_large_1: type revolute, parent JLM3915_JTLU60926_JTLU60926_JTLU60926_JTLU60926_JTLU60926_JTLU60926_JTLU60926_JTLU60926_JTLU60926_U_tj_out, child JLM3915_JTLU60926_JTLU60926_JTLU60926_JTLU60926_JTLU60926_JTLU60926_JTLU60926_JTLU60926_JTLU60926_U_tj_body, origin xyz=0.0 0.0 0.0 rpy=0.0 0.0 3.141592653589793, axis 0 0 1, limit lower=-3.1416 upper=3.1416 effort=60.5 velocity=0.33
- added joint JLM3915_JTLU60926_JTLU60926_JTLU60926_JTLU60926_JTLU60926_JTLU60926_JTLU60926_JTLU60926_JTLU60926_U_tj_large_2: type fixed, parent JLM3915_JTLU60926_JTLU60926_JTLU60926_JTLU60926_JTLU60926_JTLU60926_JTLU60926_JTLU60926_JTLU60926_U_tj_body, child JLM3915_JTLU60926_JTLU60926_JTLU60926_JTLU60926_JTLU60926_JTLU60926_JTLU60926_JTLU60926_JTLU60926_U_tj_in, origin xyz=-0.057 0 -0.0735 rpy=0 1.5707963267949 0, axis 0 0 0
- added joint JLM3915_JTLU60926_JTLU60926_JTLU60926_JTLU60926_JTLU60926_JTLU60926_JTLU60926_SLMU125823_U_sl_large: type fixed, parent JLM3915_JTLU60926_JTLU60926_JTLU60926_JTLU60926_JTLU60926_JTLU60926_JTLU60926_JTLU60926_ILU174537_U_ci_in, child JLM3915_JTLU60926_JTLU60926_JTLU60926_JTLU60926_JTLU60926_JTLU60926_JTLU60926_SLMU125823_U_sl_body, origin xyz=0.0 0.0 0.0 rpy=0.0 0.0 3.141592653589793, axis 0 0 0
- added joint JLM3915_JTLU60926_JTLU60926_JTLU60926_JTLU60926_JTLU60926_JTLU60926_JTLU60926_SLMU125823_U_sl_medium: type fixed, parent JLM3915_JTLU60926_JTLU60926_JTLU60926_JTLU60926_JTLU60926_JTLU60926_JTLU60926_SLMU125823_U_sl_body, child JLM3915_JTLU60926_JTLU60926_JTLU60926_JTLU60926_JTLU60926_JTLU60926_IMU127902_reverse_IMU127902_U_ic_in, origin xyz=0 0 -0.2 rpy=3.14159265358979 0 0, axis 0 0 0
- added joint JLM3915_JTLU60926_JTLU60926_JTLU60926_SLMU125824_U_sl_large: type fixed, parent JLM3915_JTLU60926_JTLU60926_JTLU60926_JTLU60926_ILU174538_U_ci_in, child JLM3915_JTLU60926_JTLU60926_JTLU60926_SLMU125824_U_sl_body, origin xyz=0.0 0.0 0.0 rpy=0.0 0.0 3.141592653589793, axis 0 0 0
- added joint JLM3915_JTLU60926_JTLU60926_JTLU60926_SLMU125824_U_sl_medium: type fixed, parent JLM3915_JTLU60926_JTLU60926_JTLU60926_SLMU125824_U_sl_body, child JLM3915_JTLU60926_JTLU60926_IMU127903_reverse_IMU127903_U_ic_in, origin xyz=0 0 -0.2 rpy=3.14159265358979 0 0, axis 0 0 0

Commit message: 🐞 fix(RL 环境): pybullet的底层输出
屏蔽掉了pybullet的底层输出

File: src/RobotConfigDesignEnv/robotConfigDesign/res/rebot.urdf (robot description, URDF)
Before this commit: robot UNNAMED_47, 25 links, 24 joints
Links:
- removed link BLM57_BLU858_BLU858_BLU858_BLU858_BLU858_BLU858_BLU858_BLU858_BLU858_BLU858_BLU858_BLU858_BLU858_U_b_body
- removed link BLM57_BLU858_BLU858_BLU858_BLU858_BLU858_BLU858_BLU858_BLU858_BLU858_BLU858_BLU858_BLU858_BLU858_U_b_in
- removed link BLM57_BLU858_BLU858_BLU858_BLU858_BLU858_BLU858_BLU858_BLU858_BLU858_BLU858_BLU858_BLU858_ILU1732_U_ci_body
- removed link BLM57_BLU858_BLU858_BLU858_BLU858_BLU858_BLU858_BLU858_BLU858_BLU858_BLU858_BLU858_BLU858_ILU1732_U_ci_in
- removed link BLM57_BLU858_BLU858_BLU858_BLU858_BLU858_BLU858_BLU858_BLU858_BLU858_BLU858_BLU858_JTLU600_U_tj_body
- removed link BLM57_BLU858_BLU858_BLU858_BLU858_BLU858_BLU858_BLU858_BLU858_BLU858_BLU858_BLU858_JTLU600_U_tj_in
- removed link BLM57_BLU858_BLU858_BLU858_BLU858_BLU858_BLU858_BLU858_BLU858_BLU858_BLU858_ILU1733_U_ci_body
- removed link BLM57_BLU858_BLU858_BLU858_BLU858_BLU858_BLU858_BLU858_BLU858_BLU858_BLU858_ILU1733_U_ci_in
- removed link BLM57_BLU858_BLU858_BLU858_BLU858_BLU858_BLU858_BLU858_BLU858_BLU858_SLU366_U_sl_body
- removed link BLM57_BLU858_BLU858_BLU858_BLU858_BLU858_BLU858_BLU858_BLU858_ILU1734_U_reverse_U_ci_body
- removed link BLM57_BLU858_BLU858_BLU858_BLU858_BLU858_BLU858_BLU858_BLU858_ILU1734_U_reverse_U_ci_in
- removed link BLM57_BLU858_BLU858_BLU858_BLU858_BLU858_BLU858_BLU858_CLMU247_U_reverse_U_cl_body
- removed link BLM57_BLU858_BLU858_BLU858_BLU858_BLU858_BLU858_BLU858_CLMU247_U_reverse_U_cl_in_1
- removed link BLM57_BLU858_BLU858_BLU858_BLU858_BLU858_BLU858_BLU858_CLMU247_U_reverse_U_cl_in_2
- removed link BLM57_BLU858_BLU858_BLU858_BLU858_BLU858_BLU858_IMU1172_reverse_IMU1172_U_reverse_U_ic_body
- removed link BLM57_BLU858_BLU858_BLU858_BLU858_BLU858_BLU858_IMU1172_reverse_IMU1172_U_reverse_U_ic_in
- removed link BLM57_BLU858_BLU858_BLU858_BLU858_BLU858_SMSU336_U_sl_body
- removed link BLM57_BLU858_BLU858_BLU858_BLU858_ISU288_U_reverse_U_ic_body
- removed link BLM57_BLU858_BLU858_BLU858_BLU858_ISU288_U_reverse_U_ic_in
- removed link BLM57_BLU858_BLU858_BLU858_JSU192_U_reverse_U_tj_body
- removed link BLM57_BLU858_BLU858_BLU858_JSU192_U_reverse_U_tj_in
- removed link BLM57_BLU858_BLU858_ISU289_reverse_ISU289_U_ic_body
- removed link BLM57_BLU858_BLU858_ISU289_reverse_ISU289_U_ic_in
- removed link BLM57_BLU858_ESU84_U_ee_body
- removed link BLM57_BLU858_ESU84_U_ee_in
- added link BLM2_BLU58_BLU58_BLU58_BLU58_BLU58_BLU58_BLU58_U_b_body, mass 1; collision mesh filename=package://base-l.SLDASM/meshes/b_body.STL; visual mesh filename=package://base-l.SLDASM/meshes/b_body.STL
- added link BLM2_BLU58_BLU58_BLU58_BLU58_BLU58_BLU58_BLU58_U_b_in, mass 5.9754; collision mesh filename=package://base-l.SLDASM/meshes/b_in.STL; visual mesh filename=package://base-l.SLDASM/meshes/b_in.STL
- added link BLM2_BLU58_BLU58_BLU58_BLU58_BLU58_BLU58_ILU189_U_ci_body, mass 0; collision mesh filename=package://input_connector_l.SLDASM/meshes/ci_body.STL; visual mesh filename=package://input_connector_l.SLDASM/meshes/ci_body.STL
- added link BLM2_BLU58_BLU58_BLU58_BLU58_BLU58_BLU58_ILU189_U_ci_in, mass 0; collision mesh filename=package://input_connector_l.SLDASM/meshes/ci_in.STL; visual mesh filename=package://input_connector_l.SLDASM/meshes/ci_in.STL
- added link BLM2_BLU58_BLU58_BLU58_BLU58_BLU58_SLU54_U_sl_body, mass 0.42412; collision mesh filename=package://straight_link-l.SLDASM/meshes/sl_body.STL; visual mesh filename=package://straight_link-l.SLDASM/meshes/sl_body.STL
- added link BLM2_BLU58_BLU58_BLU58_BLU58_ILU190_U_reverse_U_ci_body, mass 0; collision mesh filename=package://input_connector_l.SLDASM/meshes/ci_body.STL; visual mesh filename=package://input_connector_l.SLDASM/meshes/ci_body.STL
- added link BLM2_BLU58_BLU58_BLU58_BLU58_ILU190_U_reverse_U_ci_in, mass 0; collision mesh filename=package://input_connector_l.SLDASM/meshes/ci_in.STL; visual mesh filename=package://input_connector_l.SLDASM/meshes/ci_in.STL
- added link BLM2_BLU58_BLU58_BLU58_JTLU82_U_reverse_U_tj_body, mass 1.5884; collision mesh filename=package://jointT-l.SLDASM/meshes/tj_body.STL; visual mesh filename=package://jointT-l.SLDASM/meshes/tj_body.STL
- added link BLM2_BLU58_BLU58_BLU58_JTLU82_U_reverse_U_tj_in, mass 1.5884; collision mesh filename=package://jointT-l.SLDASM/meshes/tj_in.STL; visual mesh filename=package://jointT-l.SLDASM/meshes/tj_in.STL
- added link BLM2_BLU58_BLU58_ILU191_reverse_ILU191_U_ci_body, mass 0; collision mesh filename=package://input_connector_l.SLDASM/meshes/ci_body.STL; visual mesh filename=package://input_connector_l.SLDASM/meshes/ci_body.STL
- added link BLM2_BLU58_BLU58_ILU191_reverse_ILU191_U_ci_in, mass 0; collision mesh filename=package://input_connector_l.SLDASM/meshes/ci_in.STL; visual mesh filename=package://input_connector_l.SLDASM/meshes/ci_in.STL
- added link BLM2_BLU58_ELU6_U_ee_body, mass 0.05413; collision mesh filename=package://end_effector_v_l.SLDASM/meshes/ee_body.STL; visual mesh filename=package://end_effector_v_l.SLDASM/meshes/ee_body.STL
- added link BLM2_BLU58_ELU6_U_ee_in, mass 0; collision mesh filename=package://end_effector_v_l.SLDASM/meshes/ee_in.STL; visual mesh filename=package://end_effector_v_l.SLDASM/meshes/ee_in.STL
Joints:
- removed joint BLM57_BLU858_BLU858_BLU858_BLU858_BLU858_BLU858_BLU858_BLU858_BLU858_BLU858_BLU858_BLU858_BLU858_U_b_large
- removed joint BLM57_BLU858_BLU858_BLU858_BLU858_BLU858_BLU858_BLU858_BLU858_BLU858_BLU858_BLU858_BLU858_ILU1732_U_ci_large_1
- removed joint BLM57_BLU858_BLU858_BLU858_BLU858_BLU858_BLU858_BLU858_BLU858_BLU858_BLU858_BLU858_BLU858_ILU1732_U_ci_large_2
- removed joint BLM57_BLU858_BLU858_BLU858_BLU858_BLU858_BLU858_BLU858_BLU858_BLU858_BLU858_BLU858_JTLU600_U_tj_large_1
- removed joint BLM57_BLU858_BLU858_BLU858_BLU858_BLU858_BLU858_BLU858_BLU858_BLU858_BLU858_BLU858_JTLU600_U_tj_large_2
- removed joint BLM57_BLU858_BLU858_BLU858_BLU858_BLU858_BLU858_BLU858_BLU858_BLU858_BLU858_ILU1733_U_ci_large_1
- removed joint BLM57_BLU858_BLU858_BLU858_BLU858_BLU858_BLU858_BLU858_BLU858_BLU858_BLU858_ILU1733_U_ci_large_2
- removed joint BLM57_BLU858_BLU858_BLU858_BLU858_BLU858_BLU858_BLU858_BLU858_BLU858_SLU366_U_sl_large_1
- removed joint BLM57_BLU858_BLU858_BLU858_BLU858_BLU858_BLU858_BLU858_BLU858_BLU858_SLU366_U_sl_large_2
- removed joint BLM57_BLU858_BLU858_BLU858_BLU858_BLU858_BLU858_BLU858_BLU858_ILU1734_U_reverse_U_ci_large_1
- removed joint BLM57_BLU858_BLU858_BLU858_BLU858_BLU858_BLU858_BLU858_BLU858_ILU1734_U_reverse_U_ci_large_2
- removed joint BLM57_BLU858_BLU858_BLU858_BLU858_BLU858_BLU858_BLU858_CLMU247_U_reverse_U_cl_large
- removed joint BLM57_BLU858_BLU858_BLU858_BLU858_BLU858_BLU858_BLU858_CLMU247_U_reverse_U_cl_medium
- removed joint BLM57_BLU858_BLU858_BLU858_BLU858_BLU858_BLU858_IMU1172_reverse_IMU1172_U_reverse_U_ic_medium_1
- removed joint BLM57_BLU858_BLU858_BLU858_BLU858_BLU858_BLU858_IMU1172_reverse_IMU1172_U_reverse_U_ic_medium_2
- removed joint BLM57_BLU858_BLU858_BLU858_BLU858_BLU858_SMSU336_U_sl_medium
- removed joint BLM57_BLU858_BLU858_BLU858_BLU858_BLU858_SMSU336_U_sl_small
- removed joint BLM57_BLU858_BLU858_BLU858_BLU858_ISU288_U_reverse_U_ic_small_1
- removed joint BLM57_BLU858_BLU858_BLU858_BLU858_ISU288_U_reverse_U_ic_small_2
- removed joint BLM57_BLU858_BLU858_BLU858_JSU192_U_reverse_U_tj_small_1
- removed joint BLM57_BLU858_BLU858_BLU858_JSU192_U_reverse_U_tj_small_2
- removed joint BLM57_BLU858_BLU858_ISU289_reverse_ISU289_U_ic_small_1
- removed joint BLM57_BLU858_BLU858_ISU289_reverse_ISU289_U_ic_small_2
- removed joint BLM57_BLU858_ESU84_U_ee_small
- added joint BLM2_BLU58_BLU58_BLU58_BLU58_BLU58_BLU58_BLU58_U_b_large: type fixed, parent BLM2_BLU58_BLU58_BLU58_BLU58_BLU58_BLU58_BLU58_U_b_body, child BLM2_BLU58_BLU58_BLU58_BLU58_BLU58_BLU58_BLU58_U_b_in, origin xyz=0 0 0.0513 rpy=3.14159265358979 0 0, axis 0 0 1
- added joint BLM2_BLU58_BLU58_BLU58_BLU58_BLU58_BLU58_ILU189_U_ci_large_1: type fixed, parent BLM2_BLU58_BLU58_BLU58_BLU58_BLU58_BLU58_BLU58_U_b_in, child BLM2_BLU58_BLU58_BLU58_BLU58_BLU58_BLU58_ILU189_U_ci_body, origin xyz=0 0 0 rpy=0 0 0, axis 0 0 0
- added joint BLM2_BLU58_BLU58_BLU58_BLU58_BLU58_BLU58_ILU189_U_ci_large_2: type fixed, parent BLM2_BLU58_BLU58_BLU58_BLU58_BLU58_BLU58_ILU189_U_ci_body, child BLM2_BLU58_BLU58_BLU58_BLU58_BLU58_BLU58_ILU189_U_ci_in, origin xyz=0 0 -0.0114 rpy=0 0 0, axis 0 0 0
- added joint BLM2_BLU58_BLU58_BLU58_BLU58_BLU58_SLU54_U_sl_large_1: type fixed, parent BLM2_BLU58_BLU58_BLU58_BLU58_BLU58_BLU58_ILU189_U_ci_in, child BLM2_BLU58_BLU58_BLU58_BLU58_BLU58_SLU54_U_sl_body, origin xyz=0 0 0 rpy=0 0 0, axis 0 0 0
- added joint BLM2_BLU58_BLU58_BLU58_BLU58_BLU58_SLU54_U_sl_large_2: type fixed, parent BLM2_BLU58_BLU58_BLU58_BLU58_BLU58_SLU54_U_sl_body, child BLM2_BLU58_BLU58_BLU58_BLU58_ILU190_U_reverse_U_ci_in, origin xyz=0 0 -0.15 rpy=3.14159265358979 0 0, axis 0 0 0
- added joint BLM2_BLU58_BLU58_BLU58_BLU58_ILU190_U_reverse_U_ci_large_1: type fixed, parent BLM2_BLU58_BLU58_BLU58_BLU58_ILU190_U_reverse_U_ci_body, child BLM2_BLU58_BLU58_BLU58_JTLU82_U_reverse_U_tj_in, origin xyz=-0.0 -0.0 -0.0 rpy=0.0 0.0 0.0, axis 0 0 0
- added joint BLM2_BLU58_BLU58_BLU58_BLU58_ILU190_U_reverse_U_ci_large_2: type fixed, parent BLM2_BLU58_BLU58_BLU58_BLU58_ILU190_U_reverse_U_ci_in, child BLM2_BLU58_BLU58_BLU58_BLU58_ILU190_U_reverse_U_ci_body, origin xyz=0.0 0.0 0.0114 rpy=0.0 0.0 3.141592653589793, axis 0 0 0
- added joint BLM2_BLU58_BLU58_BLU58_JTLU82_U_reverse_U_tj_large_1: type revolute, parent BLM2_BLU58_BLU58_BLU58_JTLU82_U_reverse_U_tj_body, child BLM2_BLU58_BLU58_ILU191_reverse_ILU191_U_ci_in, origin xyz=-0.0 -0.0 -0.0 rpy=0.0 0.0 0.0, axis 0 0 1, limit lower=-3.1416 upper=3.1416 effort=60.5 velocity=0.33
- added joint BLM2_BLU58_BLU58_BLU58_JTLU82_U_reverse_U_tj_large_2: type fixed, parent BLM2_BLU58_BLU58_BLU58_JTLU82_U_reverse_U_tj_in, child BLM2_BLU58_BLU58_BLU58_JTLU82_U_reverse_U_tj_body, origin xyz=-0.0735000000000002 -0.0 0.05699999999999974 rpy=0.0 -1.5707963267949 0.0, axis 0 0 0
- added joint BLM2_BLU58_BLU58_ILU191_reverse_ILU191_U_ci_large_1: type fixed, parent BLM2_BLU58_BLU58_ILU191_reverse_ILU191_U_ci_body, child BLM2_BLU58_ELU6_U_ee_in, origin xyz=-0.0 -0.0 -0.0 rpy=0.0 0.0 0.0, axis 0 0 0
- added joint BLM2_BLU58_BLU58_ILU191_reverse_ILU191_U_ci_large_2: type fixed, parent BLM2_BLU58_BLU58_ILU191_reverse_ILU191_U_ci_in, child BLM2_BLU58_BLU58_ILU191_reverse_ILU191_U_ci_body, origin xyz=-0.0 -0.0 0.0114 rpy=0.0 0.0 0.0, axis 0 0 0
- added joint BLM2_BLU58_ELU6_U_ee_large: type fixed, parent BLM2_BLU58_ELU6_U_ee_in, child BLM2_BLU58_ELU6_U_ee_body, origin xyz=0 0 0 rpy=0 0 0, axis 0 0 0
