Commit message: ✨ feat(README):  更新README

File: src/RobotConfigDesignEnv/robotConfigDesign/res/rebot.urdf (robot description, URDF)
Before this commit: robot UNNAMED_5, 13 links, 12 joints
Links:
- removed link BLM2_BLU58_BLU58_BLU58_BLU58_BLU58_BLU58_BLU58_U_b_body
- removed link BLM2_BLU58_BLU58_BLU58_BLU58_BLU58_BLU58_BLU58_U_b_in
- removed link BLM2_BLU58_BLU58_BLU58_BLU58_BLU58_BLU58_ILU189_U_ci_body
- removed link BLM2_BLU58_BLU58_BLU58_BLU58_BLU58_BLU58_ILU189_U_ci_in
- removed link BLM2_BLU58_BLU58_BLU58_BLU58_BLU58_SLU54_U_sl_body
- removed link BLM2_BLU58_BLU58_BLU58_BLU58_ILU190_U_reverse_U_ci_body
- removed link BLM2_BLU58_BLU58_BLU58_BLU58_ILU190_U_reverse_U_ci_in
- removed link BLM2_BLU58_BLU58_BLU58_JTLU82_U_reverse_U_tj_body
- removed link BLM2_BLU58_BLU58_BLU58_JTLU82_U_reverse_U_tj_in
- removed link BLM2_BLU58_BLU58_ILU191_reverse_ILU191_U_ci_body
- removed link BLM2_BLU58_BLU58_ILU191_reverse_ILU191_U_ci_in
- removed link BLM2_BLU58_ELU6_U_ee_body
- removed link BLM2_BLU58_ELU6_U_ee_in
- added link BASEM297_BASEM0_BASEM0_BASEM0_b_body, mass 0.5; collision mesh filename=package://base-m.SLDASM/meshes/b_body.STL; visual mesh filename=package://base-m.SLDASM/meshes/b_body.STL
- added link BASEM297_BASEM0_BASEM0_BASEM0_b_in, mass 3.3499; collision mesh filename=package://base-m.SLDASM/meshes/b_in.STL; visual mesh filename=package://base-m.SLDASM/meshes/b_in.STL
- added link BASEM297_BASEM0_CONNECTORM0_CONNECTORM0_ic_body, mass 0; collision mesh filename=package://input_connector_m.SLDASM/meshes/ic_body.STL; visual mesh filename=package://input_connector_m.SLDASM/meshes/ic_body.STL
- added link BASEM297_BASEM0_CONNECTORM0_CONNECTORM0_ic_in, mass 0.50882; collision mesh filename=package://input_connector_m.SLDASM/meshes/ic_in.STL; visual mesh filename=package://input_connector_m.SLDASM/meshes/ic_in.STL
Joints:
- removed joint BLM2_BLU58_BLU58_BLU58_BLU58_BLU58_BLU58_BLU58_U_b_large
- removed joint BLM2_BLU58_BLU58_BLU58_BLU58_BLU58_BLU58_ILU189_U_ci_large_1
- removed joint BLM2_BLU58_BLU58_BLU58_BLU58_BLU58_BLU58_ILU189_U_ci_large_2
- removed joint BLM2_BLU58_BLU58_BLU58_BLU58_BLU58_SLU54_U_sl_large_1
- removed joint BLM2_BLU58_BLU58_BLU58_BLU58_BLU58_SLU54_U_sl_large_2
- removed joint BLM2_BLU58_BLU58_BLU58_BLU58_ILU190_U_reverse_U_ci_large_1
- removed joint BLM2_BLU58_BLU58_BLU58_BLU58_ILU190_U_reverse_U_ci_large_2
- removed joint BLM2_BLU58_BLU58_BLU58_JTLU82_U_reverse_U_tj_large_1
- removed joint BLM2_BLU58_BLU58_BLU58_JTLU82_U_reverse_U_tj_large_2
- removed joint BLM2_BLU58_BLU58_ILU191_reverse_ILU191_U_ci_large_1
- removed joint BLM2_BLU58_BLU58_ILU191_reverse_ILU191_U_ci_large_2
- removed joint BLM2_BLU58_ELU6_U_ee_large
- added joint BASEM297_BASEM0_BASEM0_BASEM0_b_medium: type fixed, parent BASEM297_BASEM0_BASEM0_BASEM0_b_body, child BASEM297_BASEM0_BASEM0_BASEM0_b_in, origin xyz=0 0 0.0423 rpy=3.14159265358979 0 0, axis 0 0 0
- added joint BASEM297_BASEM0_CONNECTORM0_CONNECTORM0_ic_medium_1: type fixed, parent BASEM297_BASEM0_BASEM0_BASEM0_b_in, child BASEM297_BASEM0_CONNECTORM0_CONNECTORM0_ic_body, origin xyz=0 0 0 rpy=0 0 0, axis 0 0 0
- added joint BASEM297_BASEM0_CONNECTORM0_CONNECTORM0_ic_medium_2: type fixed, parent BASEM297_BASEM0_CONNECTORM0_CONNECTORM0_ic_body, child BASEM297_BASEM0_CONNECTORM0_CONNECTORM0_ic_in, origin xyz=0 0 -0.0094 rpy=0 0 0, axis 0 0 0

Commit message: ✨ feat(RL环境): 配置文件
模块库和环境参数配置文件

File: src/RobotConfigDesignEnv/robotConfigDesign/res/rebot.urdf (robot description, URDF)
Before this commit: robot UNNAMED_199, 4 links, 3 joints
Links:
- removed link BASEM297_BASEM0_BASEM0_BASEM0_b_body
- removed link BASEM297_BASEM0_BASEM0_BASEM0_b_in
- removed link BASEM297_BASEM0_CONNECTORM0_CONNECTORM0_ic_body
- removed link BASEM297_BASEM0_CONNECTORM0_CONNECTORM0_ic_in
- added link BASEL3553_BASEL8028_BASEL8028_BASEL8028_BASEL8028_BASEL8028_BASEL8028_BASEL8028_b_body, mass 1; collision mesh filename=package://base-l.SLDASM/meshes/b_body.STL; visual mesh filename=package://base-l.SLDASM/meshes/b_body.STL
- added link BASEL3553_BASEL8028_BASEL8028_BASEL8028_BASEL8028_BASEL8028_BASEL8028_BASEL8028_b_in, mass 5.9754; collision mesh filename=package://base-l.SLDASM/meshes/b_in.STL; visual mesh filename=package://base-l.SLDASM/meshes/b_in.STL
- added link BASEL3553_BASEL8028_BASEL8028_BASEL8028_BASEL8028_BASEL8028_BASEL8028_CONNECTORL22282_ci_body, mass 0; collision mesh filename=package://input_connector_l.SLDASM/meshes/ci_body.STL; visual mesh filename=package://input_connector_l.SLDASM/meshes/ci_body.STL
- added link BASEL3553_BASEL8028_BASEL8028_BASEL8028_BASEL8028_BASEL8028_BASEL8028_CONNECTORL22282_ci_in, mass 0; collision mesh filename=package://input_connector_l.SLDASM/meshes/ci_in.STL; visual mesh filename=package://input_connector_l.SLDASM/meshes/ci_in.STL
- added link BASEL3553_BASEL8028_BASEL8028_BASEL8028_BASEL8028_BASEL8028_JOINTL3965_tj_body, mass 1.5884; collision mesh filename=package://jointT-l.SLDASM/meshes/tj_body.STL; visual mesh filename=package://jointT-l.SLDASM/meshes/tj_body.STL
- added link BASEL3553_BASEL8028_BASEL8028_BASEL8028_BASEL8028_BASEL8028_JOINTL3965_tj_in, mass 1.5884; collision mesh filename=package://jointT-l.SLDASM/meshes/tj_in.STL; visual mesh filename=package://jointT-l.SLDASM/meshes/tj_in.STL
- added link BASEL3553_BASEL8028_BASEL8028_BASEL8028_BASEL8028_CONNECTORL22283_ci_body, mass 0; collision mesh filename=package://input_connector_l.SLDASM/meshes/ci_body.STL; visual mesh filename=package://input_connector_l.SLDASM/meshes/ci_body.STL
- added link BASEL3553_BASEL8028_BASEL8028_BASEL8028_BASEL8028_CONNECTORL22283_ci_in, mass 0; collision mesh filename=package://input_connector_l.SLDASM/meshes/ci_in.STL; visual mesh filename=package://input_connector_l.SLDASM/meshes/ci_in.STL
- added link BASEL3553_BASEL8028_BASEL8028_BASEL8028_STRAIGHTLINKLM11493_sl_body, mass 1.4196; collision mesh filename=package://straight_link-lm.SLDASM/meshes/sl_body.STL; visual mesh filename=package://straight_link-lm.SLDASM/meshes/sl_body.STL
- added link BASEL3553_BASEL8028_BASEL8028_CONNECTORM24516_reverse_CONNECTORM24516_ic_body, mass 0; collision mesh filename=package://input_connector_m.SLDASM/meshes/ic_body.STL; visual mesh filename=package://input_connector_m.SLDASM/meshes/ic_body.STL
- added link BASEL3553_BASEL8028_BASEL8028_CONNECTORM24516_reverse_CONNECTORM24516_ic_in, mass 0.50882; collision mesh filename=package://input_connector_m.SLDASM/meshes/ic_in.STL; visual mesh filename=package://input_connector_m.SLDASM/meshes/ic_in.STL
- added link BASEL3553_BASEL8028_ENDEFFECTORM2500_ee_body, mass 0.0019211; collision mesh filename=package://end_effector_v_m.SLDASM/meshes/ee_body.STL; visual mesh filename=package://end_effector_v_m.SLDASM/meshes/ee_body.STL
- added link BASEL3553_BASEL8028_ENDEFFECTORM2500_ee_in, mass 0.0019211; collision mesh filename=package://end_effector_v_m.SLDASM/meshes/ee_in.STL; visual mesh filename=package://end_effector_v_m.SLDASM/meshes/ee_in.STL
Joints:
- removed joint BASEM297_BASEM0_BASEM0_BASEM0_b_medium
- removed joint BASEM297_BASEM0_CONNECTORM0_CONNECTORM0_ic_medium_1
- removed joint BASEM297_BASEM0_CONNECTORM0_CONNECTORM0_ic_medium_2
- added joint BASEL3553_BASEL8028_BASEL8028_BASEL8028_BASEL8028_BASEL8028_BASEL8028_BASEL8028_b_large: type fixed, parent BASEL3553_BASEL8028_BASEL8028_BASEL8028_BASEL8028_BASEL8028_BASEL8028_BASEL8028_b_body, child BASEL3553_BASEL8028_BASEL8028_BASEL8028_BASEL8028_BASEL8028_BASEL8028_BASEL8028_b_in, origin xyz=0 0 0.0513 rpy=3.14159265358979 0 0, axis 0 0 1
- added joint BASEL3553_BASEL8028_BASEL8028_BASEL8028_BASEL8028_BASEL8028_BASEL8028_CONNECTORL22282_ci_large_1: type fixed, parent BASEL3553_BASEL8028_BASEL8028_BASEL8028_BASEL8028_BASEL8028_BASEL8028_BASEL8028_b_in, child BASEL3553_BASEL8028_BASEL8028_BASEL8028_BASEL8028_BASEL8028_BASEL8028_CONNECTORL22282_ci_body, origin xyz=0 0 0 rpy=0 0 0, axis 0 0 0
- added joint BASEL3553_BASEL8028_BASEL8028_BASEL8028_BASEL8028_BASEL8028_BASEL8028_CONNECTORL22282_ci_large_2: type fixed, parent BASEL3553_BASEL8028_BASEL8028_BASEL8028_BASEL8028_BASEL8028_BASEL8028_CONNECTORL22282_ci_body, child BASEL3553_BASEL8028_BASEL8028_BASEL8028_BASEL8028_BASEL8028_BASEL8028_CONNECTORL22282_ci_in, origin xyz=0 0 -0.0114 rpy=0 0 0, axis 0 0 0
- added joint BASEL3553_BASEL8028_BASEL8028_BASEL8028_BASEL8028_BASEL8028_JOINTL3965_tj_large_1: type revolute, parent BASEL3553_BASEL8028_BASEL8028_BASEL8028_BASEL8028_BASEL8028_BASEL8028_CONNECTORL22282_ci_in, child BASEL3553_BASEL8028_BASEL8028_BASEL8028_BASEL8028_BASEL8028_JOINTL3965_tj_body, origin xyz=0.0 0.0 0.0 rpy=0.0 0.0 3.141592653589793, axis 0 0 1, limit lower=-3.1416 upper=3.1416 effort=60.5 velocity=0.33
- added joint BASEL3553_BASEL8028_BASEL8028_BASEL8028_BASEL8028_BASEL8028_JOINTL3965_tj_large_2: type fixed, parent BASEL3553_BASEL8028_BASEL8028_BASEL8028_BASEL8028_BASEL8028_JOINTL3965_tj_body, child BASEL3553_BASEL8028_BASEL8028_BASEL8028_BASEL8028_BASEL8028_JOINTL3965_tj_in, origin xyz=-0.057 0 -0.0735 rpy=0 1.5707963267949 0, axis 0 0 0
- added joint BASEL3553_BASEL8028_BASEL8028_BASEL8028_BASEL8028_CONNECTORL22283_ci_large_1: type fixed, parent BASEL3553_BASEL8028_BASEL8028_BASEL8028_BASEL8028_BASEL8028_JOINTL3965_tj_in, child BASEL3553_BASEL8028_BASEL8028_BASEL8028_BASEL8028_CONNECTORL22283_ci_body, origin xyz=0 0 0 rpy=0 0 0, axis 0 0 0
- added joint BASEL3553_BASEL8028_BASEL8028_BASEL8028_BASEL8028_CONNECTORL22283_ci_large_2: type fixed, parent BASEL3553_BASEL8028_BASEL8028_BASEL8028_BASEL8028_CONNECTORL22283_ci_body, child BASEL3553_BASEL8028_BASEL8028_BASEL8028_BASEL8028_CONNECTORL22283_ci_in, origin xyz=0 0 -0.0114 rpy=0 0 0, axis 0 0 0
- added joint BASEL3553_BASEL8028_BASEL8028_BASEL8028_STRAIGHTLINKLM11493_sl_large: type fixed, parent BASEL3553_BASEL8028_BASEL8028_BASEL8028_BASEL8028_CONNECTORL22283_ci_in, child BASEL3553_BASEL8028_BASEL8028_BASEL8028_STRAIGHTLINKLM11493_sl_body, origin xyz=0.0 0.0 0.0 rpy=0.0 0.0 3.141592653589793, axis 0 0 0
- added joint BASEL3553_BASEL8028_BASEL8028_BASEL8028_STRAIGHTLINKLM11493_sl_medium: type fixed, parent BASEL3553_BASEL8028_BASEL8028_BASEL8028_STRAIGHTLINKLM11493_sl_body, child BASEL3553_BASEL8028_BASEL8028_CONNECTORM24516_reverse_CONNECTORM24516_ic_in, origin xyz=0 0 -0.2 rpy=3.14159265358979 0 0, axis 0 0 0
- added joint BASEL3553_BASEL8028_BASEL8028_CONNECTORM24516_reverse_CONNECTORM24516_ic_medium_1: type fixed, parent BASEL3553_BASEL8028_BASEL8028_CONNECTORM24516_reverse_CONNECTORM24516_ic_body, child BASEL3553_BASEL8028_ENDEFFECTORM2500_ee_in, origin xyz=-0.0 -0.0 -0.0 rpy=0.0 0.0 0.0, axis 0 0 0
- added joint BASEL3553_BASEL8028_BASEL8028_CONNECTORM24516_reverse_CONNECTORM24516_ic_medium_2: type fixed, parent BASEL3553_BASEL8028_BASEL8028_CONNECTORM24516_reverse_CONNECTORM24516_ic_in, child BASEL3553_BASEL8028_BASEL8028_CONNECTORM24516_reverse_CONNECTORM24516_ic_body, origin xyz=-0.0 -0.0 0.0094 rpy=0.0 0.0 0.0, axis 0 0 0
- added joint BASEL3553_BASEL8028_ENDEFFECTORM2500_ee_medium: type fixed, parent BASEL3553_BASEL8028_ENDEFFECTORM2500_ee_in, child BASEL3553_BASEL8028_ENDEFFECTORM2500_ee_body, origin xyz=0 0 0 rpy=0 0 0, axis 0 0 0

Commit message: 服务器上跑跑看

File: src/RobotConfigDesignEnv/robotConfigDesign/res/rebot.urdf (robot description, URDF)
Before this commit: robot UNNAMED_193, 13 links, 12 joints
Links:
- removed link BASEL3553_BASEL8028_BASEL8028_BASEL8028_BASEL8028_BASEL8028_BASEL8028_BASEL8028_b_body
- removed link BASEL3553_BASEL8028_BASEL8028_BASEL8028_BASEL8028_BASEL8028_BASEL8028_BASEL8028_b_in
- removed link BASEL3553_BASEL8028_BASEL8028_BASEL8028_BASEL8028_BASEL8028_BASEL8028_CONNECTORL22282_ci_body
- removed link BASEL3553_BASEL8028_BASEL8028_BASEL8028_BASEL8028_BASEL8028_BASEL8028_CONNECTORL22282_ci_in
- removed link BASEL3553_BASEL8028_BASEL8028_BASEL8028_BASEL8028_BASEL8028_JOINTL3965_tj_body
- removed link BASEL3553_BASEL8028_BASEL8028_BASEL8028_BASEL8028_BASEL8028_JOINTL3965_tj_in
- removed link BASEL3553_BASEL8028_BASEL8028_BASEL8028_BASEL8028_CONNECTORL22283_ci_body
- removed link BASEL3553_BASEL8028_BASEL8028_BASEL8028_BASEL8028_CONNECTORL22283_ci_in
- removed link BASEL3553_BASEL8028_BASEL8028_BASEL8028_STRAIGHTLINKLM11493_sl_body
- removed link BASEL3553_BASEL8028_BASEL8028_CONNECTORM24516_reverse_CONNECTORM24516_ic_body
- removed link BASEL3553_BASEL8028_BASEL8028_CONNECTORM24516_reverse_CONNECTORM24516_ic_in
- removed link BASEL3553_BASEL8028_ENDEFFECTORM2500_ee_body
- removed link BASEL3553_BASEL8028_ENDEFFECTORM2500_ee_in
- added link BASEM4147_BASEM23594_BASEM23594_BASEM23594_BASEM23594_BASEM23594_BASEM23594_BASEM23594_b_body, mass 0.5; collision mesh filename=package://base-m.SLDASM/meshes/b_body.STL; visual mesh filename=package://base-m.SLDASM/meshes/b_body.STL
- added link BASEM4147_BASEM23594_BASEM23594_BASEM23594_BASEM23594_BASEM23594_BASEM23594_BASEM23594_b_in, mass 3.3499; collision mesh filename=package://base-m.SLDASM/meshes/b_in.STL; visual mesh filename=package://base-m.SLDASM/meshes/b_in.STL
- added link BASEM4147_BASEM23594_BASEM23594_BASEM23594_BASEM23594_BASEM23594_BASEM23594_CONNECTORM114404_ic_body, mass 0; collision mesh filename=package://input_connector_m.SLDASM/meshes/ic_body.STL; visual mesh filename=package://input_connector_m.SLDASM/meshes/ic_body.STL
- added link BASEM4147_BASEM23594_BASEM23594_BASEM23594_BASEM23594_BASEM23594_BASEM23594_CONNECTORM114404_ic_in, mass 0.50882; collision mesh filename=package://input_connector_m.SLDASM/meshes/ic_in.STL; visual mesh filename=package://input_connector_m.SLDASM/meshes/ic_in.STL
- added link BASEM4147_BASEM23594_BASEM23594_BASEM23594_BASEM23594_BASEM23594_JOINTM64603_tj_body, mass 0.93065; collision mesh filename=package://jointT-m.SLDASM/meshes/tj_body.STL; visual mesh filename=package://jointT-m.SLDASM/meshes/tj_body.STL
- added link BASEM4147_BASEM23594_BASEM23594_BASEM23594_BASEM23594_BASEM23594_JOINTM64603_tj_in, mass 0.93066; collision mesh filename=package://jointT-m.SLDASM/meshes/tj_in.STL; visual mesh filename=package://jointT-m.SLDASM/meshes/tj_in.STL
- added link BASEM4147_BASEM23594_BASEM23594_BASEM23594_BASEM23594_CONNECTORM114405_ic_body, mass 0; collision mesh filename=package://input_connector_m.SLDASM/meshes/ic_body.STL; visual mesh filename=package://input_connector_m.SLDASM/meshes/ic_body.STL
- added link BASEM4147_BASEM23594_BASEM23594_BASEM23594_BASEM23594_CONNECTORM114405_ic_in, mass 0.50882; collision mesh filename=package://input_connector_m.SLDASM/meshes/ic_in.STL; visual mesh filename=package://input_connector_m.SLDASM/meshes/ic_in.STL
- added link BASEM4147_BASEM23594_BASEM23594_BASEM23594_STRAIGHTLINKMS15785_sl_body, mass 0.86346; collision mesh filename=package://straight_link-ms.SLDASM/meshes/sl_body.STL; visual mesh filename=package://straight_link-ms.SLDASM/meshes/sl_body.STL
- added link BASEM4147_BASEM23594_BASEM23594_CONNECTORS21493_reverse_CONNECTORS21493_ic_body, mass 0; collision mesh filename=package://input_connector_s.SLDASM/meshes/ic_body.STL; visual mesh filename=package://input_connector_s.SLDASM/meshes/ic_body.STL
- added link BASEM4147_BASEM23594_BASEM23594_CONNECTORS21493_reverse_CONNECTORS21493_ic_in, mass 0.23832; collision mesh filename=package://input_connector_s.SLDASM/meshes/ic_in.STL; visual mesh filename=package://input_connector_s.SLDASM/meshes/ic_in.STL
- added link BASEM4147_BASEM23594_ENDEFFECTORS1328_ee_body, mass 0.0019211; collision mesh filename=package://end_effector_v_s.SLDASM/meshes/ee_body.STL; visual mesh filename=package://end_effector_v_s.SLDASM/meshes/ee_body.STL
- added link BASEM4147_BASEM23594_ENDEFFECTORS1328_ee_in, mass 0.0019211; collision mesh filename=package://end_effector_v_s.SLDASM/meshes/ee_in.STL; visual mesh filename=package://end_effector_v_s.SLDASM/meshes/ee_in.STL
Joints:
- removed joint BASEL3553_BASEL8028_BASEL8028_BASEL8028_BASEL8028_BASEL8028_BASEL8028_BASEL8028_b_large
- removed joint BASEL3553_BASEL8028_BASEL8028_BASEL8028_BASEL8028_BASEL8028_BASEL8028_CONNECTORL22282_ci_large_1
- removed joint BASEL3553_BASEL8028_BASEL8028_BASEL8028_BASEL8028_BASEL8028_BASEL8028_CONNECTORL22282_ci_large_2
- removed joint BASEL3553_BASEL8028_BASEL8028_BASEL8028_BASEL8028_BASEL8028_JOINTL3965_tj_large_1
- removed joint BASEL3553_BASEL8028_BASEL8028_BASEL8028_BASEL8028_BASEL8028_JOINTL3965_tj_large_2
- removed joint BASEL3553_BASEL8028_BASEL8028_BASEL8028_BASEL8028_CONNECTORL22283_ci_large_1
- removed joint BASEL3553_BASEL8028_BASEL8028_BASEL8028_BASEL8028_CONNECTORL22283_ci_large_2
- removed joint BASEL3553_BASEL8028_BASEL8028_BASEL8028_STRAIGHTLINKLM11493_sl_large
- removed joint BASEL3553_BASEL8028_BASEL8028_BASEL8028_STRAIGHTLINKLM11493_sl_medium
- removed joint BASEL3553_BASEL8028_BASEL8028_CONNECTORM24516_reverse_CONNECTORM24516_ic_medium_1
- removed joint BASEL3553_BASEL8028_BASEL8028_CONNECTORM24516_reverse_CONNECTORM24516_ic_medium_2
- removed joint BASEL3553_BASEL8028_ENDEFFECTORM2500_ee_medium
- added joint BASEM4147_BASEM23594_BASEM23594_BASEM23594_BASEM23594_BASEM23594_BASEM23594_BASEM23594_b_medium: type fixed, parent BASEM4147_BASEM23594_BASEM23594_BASEM23594_BASEM23594_BASEM23594_BASEM23594_BASEM23594_b_body, child BASEM4147_BASEM23594_BASEM23594_BASEM23594_BASEM23594_BASEM23594_BASEM23594_BASEM23594_b_in, origin xyz=0 0 0.0423 rpy=3.14159265358979 0 0, axis 0 0 0
- added joint BASEM4147_BASEM23594_BASEM23594_BASEM23594_BASEM23594_BASEM23594_BASEM23594_CONNECTORM114404_ic_medium_1: type fixed, parent BASEM4147_BASEM23594_BASEM23594_BASEM23594_BASEM23594_BASEM23594_BASEM23594_BASEM23594_b_in, child BASEM4147_BASEM23594_BASEM23594_BASEM23594_BASEM23594_BASEM23594_BASEM23594_CONNECTORM114404_ic_body, origin xyz=0 0 0 rpy=0 0 0, axis 0 0 0
- added joint BASEM4147_BASEM23594_BASEM23594_BASEM23594_BASEM23594_BASEM23594_BASEM23594_CONNECTORM114404_ic_medium_2: type fixed, parent BASEM4147_BASEM23594_BASEM23594_BASEM23594_BASEM23594_BASEM23594_BASEM23594_CONNECTORM114404_ic_body, child BASEM4147_BASEM23594_BASEM23594_BASEM23594_BASEM23594_BASEM23594_BASEM23594_CONNECTORM114404_ic_in, origin xyz=0 0 -0.0094 rpy=0 0 0, axis 0 0 0
- added joint BASEM4147_BASEM23594_BASEM23594_BASEM23594_BASEM23594_BASEM23594_JOINTM64603_tj_medium_1: type revolute, parent BASEM4147_BASEM23594_BASEM23594_BASEM23594_BASEM23594_BASEM23594_BASEM23594_CONNECTORM114404_ic_in, child BASEM4147_BASEM23594_BASEM23594_BASEM23594_BASEM23594_BASEM23594_JOINTM64603_tj_body, origin xyz=0.0 0.0 0.0 rpy=0.0 0.0 3.141592653589793, axis 0 0 1, limit lower=-3.1416 upper=3.1416 effort=25.5 velocity=0.33
- added joint BASEM4147_BASEM23594_BASEM23594_BASEM23594_BASEM23594_BASEM23594_JOINTM64603_tj_medium_2: type fixed, parent BASEM4147_BASEM23594_BASEM23594_BASEM23594_BASEM23594_BASEM23594_JOINTM64603_tj_body, child BASEM4147_BASEM23594_BASEM23594_BASEM23594_BASEM23594_BASEM23594_JOINTM64603_tj_in, origin xyz=-0.047 0 -0.0635 rpy=0 1.5707963267949 0, axis 0 -1 0
- added joint BASEM4147_BASEM23594_BASEM23594_BASEM23594_BASEM23594_CONNECTORM114405_ic_medium_1: type fixed, parent BASEM4147_BASEM23594_BASEM23594_BASEM23594_BASEM23594_BASEM23594_JOINTM64603_tj_in, child BASEM4147_BASEM23594_BASEM23594_BASEM23594_BASEM23594_CONNECTORM114405_ic_body, origin xyz=0 0 0 rpy=0 0 0, axis 0 0 0
- added joint BASEM4147_BASEM23594_BASEM23594_BASEM23594_BASEM23594_CONNECTORM114405_ic_medium_2: type fixed, parent BASEM4147_BASEM23594_BASEM23594_BASEM23594_BASEM23594_CONNECTORM114405_ic_body, child BASEM4147_BASEM23594_BASEM23594_BASEM23594_BASEM23594_CONNECTORM114405_ic_in, origin xyz=0 0 -0.0094 rpy=0 0 0, axis 0 0 0
- added joint BASEM4147_BASEM23594_BASEM23594_BASEM23594_STRAIGHTLINKMS15785_sl_medium: type fixed, parent BASEM4147_BASEM23594_BASEM23594_BASEM23594_BASEM23594_CONNECTORM114405_ic_in, child BASEM4147_BASEM23594_BASEM23594_BASEM23594_STRAIGHTLINKMS15785_sl_body, origin xyz=0 0 0 rpy=0 0 0, axis 0 0 0
- added joint BASEM4147_BASEM23594_BASEM23594_BASEM23594_STRAIGHTLINKMS15785_sl_small: type fixed, parent BASEM4147_BASEM23594_BASEM23594_BASEM23594_STRAIGHTLINKMS15785_sl_body, child BASEM4147_BASEM23594_BASEM23594_CONNECTORS21493_reverse_CONNECTORS21493_ic_in, origin xyz=0 0 -0.2 rpy=3.1416 0 0, axis 0 0 0
- added joint BASEM4147_BASEM23594_BASEM23594_CONNECTORS21493_reverse_CONNECTORS21493_ic_small_1: type fixed, parent BASEM4147_BASEM23594_BASEM23594_CONNECTORS21493_reverse_CONNECTORS21493_ic_body, child BASEM4147_BASEM23594_ENDEFFECTORS1328_ee_in, origin xyz=-0.0 -0.0 -0.0 rpy=0.0 0.0 0.0, axis 0 0 0
- added joint BASEM4147_BASEM23594_BASEM23594_CONNECTORS21493_reverse_CONNECTORS21493_ic_small_2: type fixed, parent BASEM4147_BASEM23594_BASEM23594_CONNECTORS21493_reverse_CONNECTORS21493_ic_in, child BASEM4147_BASEM23594_BASEM23594_CONNECTORS21493_reverse_CONNECTORS21493_ic_body, origin xyz=-0.0 -0.0 0.0073 rpy=0.0 0.0 0.0, axis 0 0 0
- added joint BASEM4147_BASEM23594_ENDEFFECTORS1328_ee_small: type fixed, parent BASEM4147_BASEM23594_ENDEFFECTORS1328_ee_in, child BASEM4147_BASEM23594_ENDEFFECTORS1328_ee_body, origin xyz=0 0 0 rpy=0 0 0, axis 0 0 0
