Commit message: 环境打包

File: src/RobotConfigDesignEnv/robotConfigDesign/res/rebot.urdf (robot description, URDF)
Before this commit: robot UNNAMED_224, 13 links, 12 joints
Links:
- removed link BASEM4147_BASEM23594_BASEM23594_BASEM23594_BASEM23594_BASEM23594_BASEM23594_BASEM23594_b_body
- removed link BASEM4147_BASEM23594_BASEM23594_BASEM23594_BASEM23594_BASEM23594_BASEM23594_BASEM23594_b_in
- removed link BASEM4147_BASEM23594_BASEM23594_BASEM23594_BASEM23594_BASEM23594_BASEM23594_CONNECTORM114404_ic_body
- removed link BASEM4147_BASEM23594_BASEM23594_BASEM23594_BASEM23594_BASEM23594_BASEM23594_CONNECTORM114404_ic_in
- removed link BASEM4147_BASEM23594_BASEM23594_BASEM23594_BASEM23594_BASEM23594_JOINTM64603_tj_body
- removed link BASEM4147_BASEM23594_BASEM23594_BASEM23594_BASEM23594_BASEM23594_JOINTM64603_tj_in
- removed link BASEM4147_BASEM23594_BASEM23594_BASEM23594_BASEM23594_CONNECTORM114405_ic_body
- removed link BASEM4147_BASEM23594_BASEM23594_BASEM23594_BASEM23594_CONNECTORM114405_ic_in
- removed link BASEM4147_BASEM23594_BASEM23594_BASEM23594_STRAIGHTLINKMS15785_sl_body
- removed link BASEM4147_BASEM23594_BASEM23594_CONNECTORS21493_reverse_CONNECTORS21493_ic_body
- removed link BASEM4147_BASEM23594_BASEM23594_CONNECTORS21493_reverse_CONNECTORS21493_ic_in
- removed link BASEM4147_BASEM23594_ENDEFFECTORS1328_ee_body
- removed link BASEM4147_BASEM23594_ENDEFFECTORS1328_ee_in
- added link BASEM9_BASEM312_BASEM312_BASEM312_BASEM312_BASEM312_BASEM312_BASEM312_BASEM312_BASEM312_BASEM312_BASEM312_BASEM312_BASEM312_BASEM312_BASEM312_BASEM312_BASEM312_b_body, mass 0.5; collision mesh filename=package://base-m.SLDASM/meshes/b_body.STL; visual mesh filename=package://base-m.SLDASM/meshes/b_body.STL
- added link BASEM9_BASEM312_BASEM312_BASEM312_BASEM312_BASEM312_BASEM312_BASEM312_BASEM312_BASEM312_BASEM312_BASEM312_BASEM312_BASEM312_BASEM312_BASEM312_BASEM312_BASEM312_b_in, mass 3.3499; collision mesh filename=package://base-m.SLDASM/meshes/b_in.STL; visual mesh filename=package://base-m.SLDASM/meshes/b_in.STL
- added link BASEM9_BASEM312_BASEM312_BASEM312_BASEM312_BASEM312_BASEM312_BASEM312_BASEM312_BASEM312_BASEM312_BASEM312_BASEM312_BASEM312_BASEM312_BASEM312_BASEM312_CONNECTORM1004_ic_body, mass 0; collision mesh filename=package://input_connector_m.SLDASM/meshes/ic_body.STL; visual mesh filename=package://input_connector_m.SLDASM/meshes/ic_body.STL
- added link BASEM9_BASEM312_BASEM312_BASEM312_BASEM312_BASEM312_BASEM312_BASEM312_BASEM312_BASEM312_BASEM312_BASEM312_BASEM312_BASEM312_BASEM312_BASEM312_BASEM312_CONNECTORM1004_ic_in, mass 0.50882; collision mesh filename=package://input_connector_m.SLDASM/meshes/ic_in.STL; visual mesh filename=package://input_connector_m.SLDASM/meshes/ic_in.STL
- added link BASEM9_BASEM312_BASEM312_BASEM312_BASEM312_BASEM312_BASEM312_BASEM312_BASEM312_BASEM312_BASEM312_BASEM312_BASEM312_BASEM312_BASEM312_BASEM312_JOINTM688_tj_body, mass 0.93065; collision mesh filename=package://jointT-m.SLDASM/meshes/tj_body.STL; visual mesh filename=package://jointT-m.SLDASM/meshes/tj_body.STL
- added link BASEM9_BASEM312_BASEM312_BASEM312_BASEM312_BASEM312_BASEM312_BASEM312_BASEM312_BASEM312_BASEM312_BASEM312_BASEM312_BASEM312_BASEM312_BASEM312_JOINTM688_tj_in, mass 0.93066; collision mesh filename=package://jointT-m.SLDASM/meshes/tj_in.STL; visual mesh filename=package://jointT-m.SLDASM/meshes/tj_in.STL
- added link BASEM9_BASEM312_BASEM312_BASEM312_BASEM312_BASEM312_BASEM312_BASEM312_BASEM312_BASEM312_BASEM312_BASEM312_BASEM312_BASEM312_BASEM312_CONNECTORM1005_ic_body, mass 0; collision mesh filename=package://input_connector_m.SLDASM/meshes/ic_body.STL; visual mesh filename=package://input_connector_m.SLDASM/meshes/ic_body.STL
- added link BASEM9_BASEM312_BASEM312_BASEM312_BASEM312_BASEM312_BASEM312_BASEM312_BASEM312_BASEM312_BASEM312_BASEM312_BASEM312_BASEM312_BASEM312_CONNECTORM1005_ic_in, mass 0.50882; collision mesh filename=package://input_connector_m.SLDASM/meshes/ic_in.STL; visual mesh filename=package://input_connector_m.SLDASM/meshes/ic_in.STL
- added link BASEM9_BASEM312_BASEM312_BASEM312_BASEM312_BASEM312_BASEM312_BASEM312_BASEM312_BASEM312_BASEM312_BASEM312_BASEM312_BASEM312_JOINTM689_tj_body, mass 0.93065; collision mesh filename=package://jointT-m.SLDASM/meshes/tj_body.STL; visual mesh filename=package://jointT-m.SLDASM/meshes/tj_body.STL
- added link BASEM9_BASEM312_BASEM312_BASEM312_BASEM312_BASEM312_BASEM312_BASEM312_BASEM312_BASEM312_BASEM312_BASEM312_BASEM312_BASEM312_JOINTM689_tj_in, mass 0.93066; collision mesh filename=package://jointT-m.SLDASM/meshes/tj_in.STL; visual mesh filename=package://jointT-m.SLDASM/meshes/tj_in.STL
- added link BASEM9_BASEM312_BASEM312_BASEM312_BASEM312_BASEM312_BASEM312_BASEM312_BASEM312_BASEM312_BASEM312_BASEM312_BASEM312_CONNECTORM1006_ic_body, mass 0; collision mesh filename=package://input_connector_m.SLDASM/meshes/ic_body.STL; visual mesh filename=package://input_connector_m.SLDASM/meshes/ic_body.STL
- added link BASEM9_BASEM312_BASEM312_BASEM312_BASEM312_BASEM312_BASEM312_BASEM312_BASEM312_BASEM312_BASEM312_BASEM312_BASEM312_CONNECTORM1006_ic_in, mass 0.50882; collision mesh filename=package://input_connector_m.SLDASM/meshes/ic_in.STL; visual mesh filename=package://input_connector_m.SLDASM/meshes/ic_in.STL
- added link BASEM9_BASEM312_BASEM312_BASEM312_BASEM312_BASEM312_BASEM312_BASEM312_BASEM312_BASEM312_BASEM312_BASEM312_JOINTM690_tj_body, mass 0.93065; collision mesh filename=package://jointT-m.SLDASM/meshes/tj_body.STL; visual mesh filename=package://jointT-m.SLDASM/meshes/tj_body.STL
- added link BASEM9_BASEM312_BASEM312_BASEM312_BASEM312_BASEM312_BASEM312_BASEM312_BASEM312_BASEM312_BASEM312_BASEM312_JOINTM690_tj_in, mass 0.93066; collision mesh filename=package://jointT-m.SLDASM/meshes/tj_in.STL; visual mesh filename=package://jointT-m.SLDASM/meshes/tj_in.STL
- added link BASEM9_BASEM312_BASEM312_BASEM312_BASEM312_BASEM312_BASEM312_BASEM312_BASEM312_BASEM312_BASEM312_CONNECTORM1007_ic_body, mass 0; collision mesh filename=package://input_connector_m.SLDASM/meshes/ic_body.STL; visual mesh filename=package://input_connector_m.SLDASM/meshes/ic_body.STL
- added link BASEM9_BASEM312_BASEM312_BASEM312_BASEM312_BASEM312_BASEM312_BASEM312_BASEM312_BASEM312_BASEM312_CONNECTORM1007_ic_in, mass 0.50882; collision mesh filename=package://input_connector_m.SLDASM/meshes/ic_in.STL; visual mesh filename=package://input_connector_m.SLDASM/meshes/ic_in.STL
- added link BASEM9_BASEM312_BASEM312_BASEM312_BASEM312_BASEM312_BASEM312_BASEM312_BASEM312_BASEM312_STRAIGHTLINKMS100_sl_body, mass 0.86346; collision mesh filename=package://straight_link-ms.SLDASM/meshes/sl_body.STL; visual mesh filename=package://straight_link-ms.SLDASM/meshes/sl_body.STL
- added link BASEM9_BASEM312_BASEM312_BASEM312_BASEM312_BASEM312_BASEM312_BASEM312_BASEM312_CONNECTORS144_reverse_ic_body, mass 0; collision mesh filename=package://input_connector_s.SLDASM/meshes/ic_body.STL; visual mesh filename=package://input_connector_s.SLDASM/meshes/ic_body.STL
- added link BASEM9_BASEM312_BASEM312_BASEM312_BASEM312_BASEM312_BASEM312_BASEM312_BASEM312_CONNECTORS144_reverse_ic_in, mass 0.23832; collision mesh filename=package://input_connector_s.SLDASM/meshes/ic_in.STL; visual mesh filename=package://input_connector_s.SLDASM/meshes/ic_in.STL
- added link BASEM9_BASEM312_BASEM312_BASEM312_BASEM312_BASEM312_BASEM312_BASEM312_JOINTS140_reverse_tj_body, mass 0.50441; collision mesh filename=package://jointT-s.SLDASM/meshes/tj_body.STL; visual mesh filename=package://jointT-s.SLDASM/meshes/tj_body.STL
- added link BASEM9_BASEM312_BASEM312_BASEM312_BASEM312_BASEM312_BASEM312_BASEM312_JOINTS140_reverse_tj_in, mass 0.50441; collision mesh filename=package://jointT-s.SLDASM/meshes/tj_in.STL; visual mesh filename=package://jointT-s.SLDASM/meshes/tj_in.STL
- added link BASEM9_BASEM312_BASEM312_BASEM312_BASEM312_BASEM312_BASEM312_CONNECTORS145_reverse_ic_body, mass 0; collision mesh filename=package://input_connector_s.SLDASM/meshes/ic_body.STL; visual mesh filename=package://input_connector_s.SLDASM/meshes/ic_body.STL
- added link BASEM9_BASEM312_BASEM312_BASEM312_BASEM312_BASEM312_BASEM312_CONNECTORS145_reverse_ic_in, mass 0.23832; collision mesh filename=package://input_connector_s.SLDASM/meshes/ic_in.STL; visual mesh filename=package://input_connector_s.SLDASM/meshes/ic_in.STL
- added link BASEM9_BASEM312_BASEM312_BASEM312_BASEM312_BASEM312_JOINTS141_reverse_tj_body, mass 0.50441; collision mesh filename=package://jointT-s.SLDASM/meshes/tj_body.STL; visual mesh filename=package://jointT-s.SLDASM/meshes/tj_body.STL
- added link BASEM9_BASEM312_BASEM312_BASEM312_BASEM312_BASEM312_JOINTS141_reverse_tj_in, mass 0.50441; collision mesh filename=package://jointT-s.SLDASM/meshes/tj_in.STL; visual mesh filename=package://jointT-s.SLDASM/meshes/tj_in.STL
- added link BASEM9_BASEM312_BASEM312_BASEM312_BASEM312_CONNECTORS146_reverse_ic_body, mass 0; collision mesh filename=package://input_connector_s.SLDASM/meshes/ic_body.STL; visual mesh filename=package://input_connector_s.SLDASM/meshes/ic_body.STL
- added link BASEM9_BASEM312_BASEM312_BASEM312_BASEM312_CONNECTORS146_reverse_ic_in, mass 0.23832; collision mesh filename=package://input_connector_s.SLDASM/meshes/ic_in.STL; visual mesh filename=package://input_connector_s.SLDASM/meshes/ic_in.STL
- added link BASEM9_BASEM312_BASEM312_BASEM312_JOINTS142_reverse_tj_body, mass 0.50441; collision mesh filename=package://jointT-s.SLDASM/meshes/tj_body.STL; visual mesh filename=package://jointT-s.SLDASM/meshes/tj_body.STL
- added link BASEM9_BASEM312_BASEM312_BASEM312_JOINTS142_reverse_tj_in, mass 0.50441; collision mesh filename=package://jointT-s.SLDASM/meshes/tj_in.STL; visual mesh filename=package://jointT-s.SLDASM/meshes/tj_in.STL
- added link BASEM9_BASEM312_BASEM312_CONNECTORS147_reverse_CONNECTORS147_ic_body, mass 0; collision mesh filename=package://input_connector_s.SLDASM/meshes/ic_body.STL; visual mesh filename=package://input_connector_s.SLDASM/meshes/ic_body.STL
- added link BASEM9_BASEM312_BASEM312_CONNECTORS147_reverse_CONNECTORS147_ic_in, mass 0.23832; collision mesh filename=package://input_connector_s.SLDASM/meshes/ic_in.STL; visual mesh filename=package://input_connector_s.SLDASM/meshes/ic_in.STL
- added link BASEM9_BASEM312_ENDEFFECTORS4_ee_body, mass 0.0019211; collision mesh filename=package://end_effector_v_s.SLDASM/meshes/ee_body.STL; visual mesh filename=package://end_effector_v_s.SLDASM/meshes/ee_body.STL
- added link BASEM9_BASEM312_ENDEFFECTORS4_ee_in, mass 0.0019211; collision mesh filename=package://end_effector_v_s.SLDASM/meshes/ee_in.STL; visual mesh filename=package://end_effector_v_s.SLDASM/meshes/ee_in.STL
Joints:
- removed joint BASEM4147_BASEM23594_BASEM23594_BASEM23594_BASEM23594_BASEM23594_BASEM23594_BASEM23594_b_medium
- removed joint BASEM4147_BASEM23594_BASEM23594_BASEM23594_BASEM23594_BASEM23594_BASEM23594_CONNECTORM114404_ic_medium_1
- removed joint BASEM4147_BASEM23594_BASEM23594_BASEM23594_BASEM23594_BASEM23594_BASEM23594_CONNECTORM114404_ic_medium_2
- removed joint BASEM4147_BASEM23594_BASEM23594_BASEM23594_BASEM23594_BASEM23594_JOINTM64603_tj_medium_1
- removed joint BASEM4147_BASEM23594_BASEM23594_BASEM23594_BASEM23594_BASEM23594_JOINTM64603_tj_medium_2
- removed joint BASEM4147_BASEM23594_BASEM23594_BASEM23594_BASEM23594_CONNECTORM114405_ic_medium_1
- removed joint BASEM4147_BASEM23594_BASEM23594_BASEM23594_BASEM23594_CONNECTORM114405_ic_medium_2
- removed joint BASEM4147_BASEM23594_BASEM23594_BASEM23594_STRAIGHTLINKMS15785_sl_medium
- removed joint BASEM4147_BASEM23594_BASEM23594_BASEM23594_STRAIGHTLINKMS15785_sl_small
- removed joint BASEM4147_BASEM23594_BASEM23594_CONNECTORS21493_reverse_CONNECTORS21493_ic_small_1
- removed joint BASEM4147_BASEM23594_BASEM23594_CONNECTORS21493_reverse_CONNECTORS21493_ic_small_2
- removed joint BASEM4147_BASEM23594_ENDEFFECTORS1328_ee_small
- added joint BASEM9_BASEM312_BASEM312_BASEM312_BASEM312_BASEM312_BASEM312_BASEM312_BASEM312_BASEM312_BASEM312_BASEM312_BASEM312_BASEM312_BASEM312_BASEM312_BASEM312_BASEM312_b_medium: type fixed, parent BASEM9_BASEM312_BASEM312_BASEM312_BASEM312_BASEM312_BASEM312_BASEM312_BASEM312_BASEM312_BASEM312_BASEM312_BASEM312_BASEM312_BASEM312_BASEM312_BASEM312_BASEM312_b_body, child BASEM9_BASEM312_BASEM312_BASEM312_BASEM312_BASEM312_BASEM312_BASEM312_BASEM312_BASEM312_BASEM312_BASEM312_BASEM312_BASEM312_BASEM312_BASEM312_BASEM312_BASEM312_b_in, origin xyz=0 0 0.0423 rpy=3.14159265358979 0 0, axis 0 0 0
- added joint BASEM9_BASEM312_BASEM312_BASEM312_BASEM312_BASEM312_BASEM312_BASEM312_BASEM312_BASEM312_BASEM312_BASEM312_BASEM312_BASEM312_BASEM312_BASEM312_BASEM312_CONNECTORM1004_ic_medium_1: type fixed, parent BASEM9_BASEM312_BASEM312_BASEM312_BASEM312_BASEM312_BASEM312_BASEM312_BASEM312_BASEM312_BASEM312_BASEM312_BASEM312_BASEM312_BASEM312_BASEM312_BASEM312_BASEM312_b_in, child BASEM9_BASEM312_BASEM312_BASEM312_BASEM312_BASEM312_BASEM312_BASEM312_BASEM312_BASEM312_BASEM312_BASEM312_BASEM312_BASEM312_BASEM312_BASEM312_BASEM312_CONNECTORM1004_ic_body, origin xyz=0 0 0 rpy=0 0 0, axis 0 0 0
- added joint BASEM9_BASEM312_BASEM312_BASEM312_BASEM312_BASEM312_BASEM312_BASEM312_BASEM312_BASEM312_BASEM312_BASEM312_BASEM312_BASEM312_BASEM312_BASEM312_BASEM312_CONNECTORM1004_ic_medium_2: type fixed, parent BASEM9_BASEM312_BASEM312_BASEM312_BASEM312_BASEM312_BASEM312_BASEM312_BASEM312_BASEM312_BASEM312_BASEM312_BASEM312_BASEM312_BASEM312_BASEM312_BASEM312_CONNECTORM1004_ic_body, child BASEM9_BASEM312_BASEM312_BASEM312_BASEM312_BASEM312_BASEM312_BASEM312_BASEM312_BASEM312_BASEM312_BASEM312_BASEM312_BASEM312_BASEM312_BASEM312_BASEM312_CONNECTORM1004_ic_in, origin xyz=0 0 -0.0094 rpy=0 0 0, axis 0 0 0
- added joint BASEM9_BASEM312_BASEM312_BASEM312_BASEM312_BASEM312_BASEM312_BASEM312_BASEM312_BASEM312_BASEM312_BASEM312_BASEM312_BASEM312_BASEM312_BASEM312_JOINTM688_tj_medium_1: type revolute, parent BASEM9_BASEM312_BASEM312_BASEM312_BASEM312_BASEM312_BASEM312_BASEM312_BASEM312_BASEM312_BASEM312_BASEM312_BASEM312_BASEM312_BASEM312_BASEM312_BASEM312_CONNECTORM1004_ic_in, child BASEM9_BASEM312_BASEM312_BASEM312_BASEM312_BASEM312_BASEM312_BASEM312_BASEM312_BASEM312_BASEM312_BASEM312_BASEM312_BASEM312_BASEM312_BASEM312_JOINTM688_tj_body, origin xyz=0.0 0.0 0.0 rpy=0.0 0.0 3.141592653589793, axis 0 0 1, limit lower=-3.1416 upper=3.1416 effort=25.5 velocity=0.33
- added joint BASEM9_BASEM312_BASEM312_BASEM312_BASEM312_BASEM312_BASEM312_BASEM312_BASEM312_BASEM312_BASEM312_BASEM312_BASEM312_BASEM312_BASEM312_BASEM312_JOINTM688_tj_medium_2: type fixed, parent BASEM9_BASEM312_BASEM312_BASEM312_BASEM312_BASEM312_BASEM312_BASEM312_BASEM312_BASEM312_BASEM312_BASEM312_BASEM312_BASEM312_BASEM312_BASEM312_JOINTM688_tj_body, child BASEM9_BASEM312_BASEM312_BASEM312_BASEM312_BASEM312_BASEM312_BASEM312_BASEM312_BASEM312_BASEM312_BASEM312_BASEM312_BASEM312_BASEM312_BASEM312_JOINTM688_tj_in, origin xyz=-0.047 0 -0.0635 rpy=0 1.5707963267949 0, axis 0 -1 0
- added joint BASEM9_BASEM312_BASEM312_BASEM312_BASEM312_BASEM312_BASEM312_BASEM312_BASEM312_BASEM312_BASEM312_BASEM312_BASEM312_BASEM312_BASEM312_CONNECTORM1005_ic_medium_1: type fixed, parent BASEM9_BASEM312_BASEM312_BASEM312_BASEM312_BASEM312_BASEM312_BASEM312_BASEM312_BASEM312_BASEM312_BASEM312_BASEM312_BASEM312_BASEM312_BASEM312_JOINTM688_tj_in, child BASEM9_BASEM312_BASEM312_BASEM312_BASEM312_BASEM312_BASEM312_BASEM312_BASEM312_BASEM312_BASEM312_BASEM312_BASEM312_BASEM312_BASEM312_CONNECTORM1005_ic_body, origin xyz=0 0 0 rpy=0 0 0, axis 0 0 0
- added joint BASEM9_BASEM312_BASEM312_BASEM312_BASEM312_BASEM312_BASEM312_BASEM312_BASEM312_BASEM312_BASEM312_BASEM312_BASEM312_BASEM312_BASEM312_CONNECTORM1005_ic_medium_2: type fixed, parent BASEM9_BASEM312_BASEM312_BASEM312_BASEM312_BASEM312_BASEM312_BASEM312_BASEM312_BASEM312_BASEM312_BASEM312_BASEM312_BASEM312_BASEM312_CONNECTORM1005_ic_body, child BASEM9_BASEM312_BASEM312_BASEM312_BASEM312_BASEM312_BASEM312_BASEM312_BASEM312_BASEM312_BASEM312_BASEM312_BASEM312_BASEM312_BASEM312_CONNECTORM1005_ic_in, origin xyz=0 0 -0.0094 rpy=0 0 0, axis 0 0 0
- added joint BASEM9_BASEM312_BASEM312_BASEM312_BASEM312_BASEM312_BASEM312_BASEM312_BASEM312_BASEM312_BASEM312_BASEM312_BASEM312_BASEM312_JOINTM689_tj_medium_1: type revolute, parent BASEM9_BASEM312_BASEM312_BASEM312_BASEM312_BASEM312_BASEM312_BASEM312_BASEM312_BASEM312_BASEM312_BASEM312_BASEM312_BASEM312_BASEM312_CONNECTORM1005_ic_in, child BASEM9_BASEM312_BASEM312_BASEM312_BASEM312_BASEM312_BASEM312_BASEM312_BASEM312_BASEM312_BASEM312_BASEM312_BASEM312_BASEM312_JOINTM689_tj_body, origin xyz=0.0 0.0 0.0 rpy=0.0 0.0 3.141592653589793, axis 0 0 1, limit lower=-3.1416 upper=3.1416 effort=25.5 velocity=0.33
- added joint BASEM9_BASEM312_BASEM312_BASEM312_BASEM312_BASEM312_BASEM312_BASEM312_BASEM312_BASEM312_BASEM312_BASEM312_BASEM312_BASEM312_JOINTM689_tj_medium_2: type fixed, parent BASEM9_BASEM312_BASEM312_BASEM312_BASEM312_BASEM312_BASEM312_BASEM312_BASEM312_BASEM312_BASEM312_BASEM312_BASEM312_BASEM312_JOINTM689_tj_body, child BASEM9_BASEM312_BASEM312_BASEM312_BASEM312_BASEM312_BASEM312_BASEM312_BASEM312_BASEM312_BASEM312_BASEM312_BASEM312_BASEM312_JOINTM689_tj_in, origin xyz=-0.047 0 -0.0635 rpy=0 1.5707963267949 0, axis 0 -1 0
- added joint BASEM9_BASEM312_BASEM312_BASEM312_BASEM312_BASEM312_BASEM312_BASEM312_BASEM312_BASEM312_BASEM312_BASEM312_BASEM312_CONNECTORM1006_ic_medium_1: type fixed, parent BASEM9_BASEM312_BASEM312_BASEM312_BASEM312_BASEM312_BASEM312_BASEM312_BASEM312_BASEM312_BASEM312_BASEM312_BASEM312_BASEM312_JOINTM689_tj_in, child BASEM9_BASEM312_BASEM312_BASEM312_BASEM312_BASEM312_BASEM312_BASEM312_BASEM312_BASEM312_BASEM312_BASEM312_BASEM312_CONNECTORM1006_ic_body, origin xyz=0 0 0 rpy=0 0 0, axis 0 0 0
- added joint BASEM9_BASEM312_BASEM312_BASEM312_BASEM312_BASEM312_BASEM312_BASEM312_BASEM312_BASEM312_BASEM312_BASEM312_BASEM312_CONNECTORM1006_ic_medium_2: type fixed, parent BASEM9_BASEM312_BASEM312_BASEM312_BASEM312_BASEM312_BASEM312_BASEM312_BASEM312_BASEM312_BASEM312_BASEM312_BASEM312_CONNECTORM1006_ic_body, child BASEM9_BASEM312_BASEM312_BASEM312_BASEM312_BASEM312_BASEM312_BASEM312_BASEM312_BASEM312_BASEM312_BASEM312_BASEM312_CONNECTORM1006_ic_in, origin xyz=0 0 -0.0094 rpy=0 0 0, axis 0 0 0
- added joint BASEM9_BASEM312_BASEM312_BASEM312_BASEM312_BASEM312_BASEM312_BASEM312_BASEM312_BASEM312_BASEM312_BASEM312_JOINTM690_tj_medium_1: type revolute, parent BASEM9_BASEM312_BASEM312_BASEM312_BASEM312_BASEM312_BASEM312_BASEM312_BASEM312_BASEM312_BASEM312_BASEM312_BASEM312_CONNECTORM1006_ic_in, child BASEM9_BASEM312_BASEM312_BASEM312_BASEM312_BASEM312_BASEM312_BASEM312_BASEM312_BASEM312_BASEM312_BASEM312_JOINTM690_tj_body, origin xyz=0.0 0.0 0.0 rpy=0.0 0.0 3.141592653589793, axis 0 0 1, limit lower=-3.1416 upper=3.1416 effort=25.5 velocity=0.33
- added joint BASEM9_BASEM312_BASEM312_BASEM312_BASEM312_BASEM312_BASEM312_BASEM312_BASEM312_BASEM312_BASEM312_BASEM312_JOINTM690_tj_medium_2: type fixed, parent BASEM9_BASEM312_BASEM312_BASEM312_BASEM312_BASEM312_BASEM312_BASEM312_BASEM312_BASEM312_BASEM312_BASEM312_JOINTM690_tj_body, child BASEM9_BASEM312_BASEM312_BASEM312_BASEM312_BASEM312_BASEM312_BASEM312_BASEM312_BASEM312_BASEM312_BASEM312_JOINTM690_tj_in, origin xyz=-0.047 0 -0.0635 rpy=0 1.5707963267949 0, axis 0 -1 0
- added joint BASEM9_BASEM312_BASEM312_BASEM312_BASEM312_BASEM312_BASEM312_BASEM312_BASEM312_BASEM312_BASEM312_CONNECTORM1007_ic_medium_1: type fixed, parent BASEM9_BASEM312_BASEM312_BASEM312_BASEM312_BASEM312_BASEM312_BASEM312_BASEM312_BASEM312_BASEM312_BASEM312_JOINTM690_tj_in, child BASEM9_BASEM312_BASEM312_BASEM312_BASEM312_BASEM312_BASEM312_BASEM312_BASEM312_BASEM312_BASEM312_CONNECTORM1007_ic_body, origin xyz=0 0 0 rpy=0 0 0, axis 0 0 0
- added joint BASEM9_BASEM312_BASEM312_BASEM312_BASEM312_BASEM312_BASEM312_BASEM312_BASEM312_BASEM312_BASEM312_CONNECTORM1007_ic_medium_2: type fixed, parent BASEM9_BASEM312_BASEM312_BASEM312_BASEM312_BASEM312_BASEM312_BASEM312_BASEM312_BASEM312_BASEM312_CONNECTORM1007_ic_body, child BASEM9_BASEM312_BASEM312_BASEM312_BASEM312_BASEM312_BASEM312_BASEM312_BASEM312_BASEM312_BASEM312_CONNECTORM1007_ic_in, origin xyz=0 0 -0.0094 rpy=0 0 0, axis 0 0 0
- added joint BASEM9_BASEM312_BASEM312_BASEM312_BASEM312_BASEM312_BASEM312_BASEM312_BASEM312_BASEM312_STRAIGHTLINKMS100_sl_medium: type fixed, parent BASEM9_BASEM312_BASEM312_BASEM312_BASEM312_BASEM312_BASEM312_BASEM312_BASEM312_BASEM312_BASEM312_CONNECTORM1007_ic_in, child BASEM9_BASEM312_BASEM312_BASEM312_BASEM312_BASEM312_BASEM312_BASEM312_BASEM312_BASEM312_STRAIGHTLINKMS100_sl_body, origin xyz=0 0 0 rpy=0 0 0, axis 0 0 0
- added joint BASEM9_BASEM312_BASEM312_BASEM312_BASEM312_BASEM312_BASEM312_BASEM312_BASEM312_BASEM312_STRAIGHTLINKMS100_sl_small: type fixed, parent BASEM9_BASEM312_BASEM312_BASEM312_BASEM312_BASEM312_BASEM312_BASEM312_BASEM312_BASEM312_STRAIGHTLINKMS100_sl_body, child BASEM9_BASEM312_BASEM312_BASEM312_BASEM312_BASEM312_BASEM312_BASEM312_BASEM312_CONNECTORS144_reverse_ic_in, origin xyz=0 0 -0.2 rpy=3.1416 0 0, axis 0 0 0
- added joint BASEM9_BASEM312_BASEM312_BASEM312_BASEM312_BASEM312_BASEM312_BASEM312_BASEM312_CONNECTORS144_reverse_ic_small_1: type fixed, parent BASEM9_BASEM312_BASEM312_BASEM312_BASEM312_BASEM312_BASEM312_BASEM312_BASEM312_CONNECTORS144_reverse_ic_body, child BASEM9_BASEM312_BASEM312_BASEM312_BASEM312_BASEM312_BASEM312_BASEM312_JOINTS140_reverse_tj_in, origin xyz=-0.0 -0.0 -0.0 rpy=0.0 0.0 0.0, axis 0 0 0
- added joint BASEM9_BASEM312_BASEM312_BASEM312_BASEM312_BASEM312_BASEM312_BASEM312_BASEM312_CONNECTORS144_reverse_ic_small_2: type fixed, parent BASEM9_BASEM312_BASEM312_BASEM312_BASEM312_BASEM312_BASEM312_BASEM312_BASEM312_CONNECTORS144_reverse_ic_in, child BASEM9_BASEM312_BASEM312_BASEM312_BASEM312_BASEM312_BASEM312_BASEM312_BASEM312_CONNECTORS144_reverse_ic_body, origin xyz=0.0 0.0 0.0073 rpy=0.0 0.0 3.141592653589793, axis 0 0 0
- added joint BASEM9_BASEM312_BASEM312_BASEM312_BASEM312_BASEM312_BASEM312_BASEM312_JOINTS140_reverse_tj_small_1: type revolute, parent BASEM9_BASEM312_BASEM312_BASEM312_BASEM312_BASEM312_BASEM312_BASEM312_JOINTS140_reverse_tj_body, child BASEM9_BASEM312_BASEM312_BASEM312_BASEM312_BASEM312_BASEM312_CONNECTORS145_reverse_ic_in, origin xyz=-0.0 -0.0 -0.0 rpy=0.0 0.0 0.0, axis 0 0 1, limit lower=-3.1416 upper=3.1416 effort=4.5 velocity=0.4
- added joint BASEM9_BASEM312_BASEM312_BASEM312_BASEM312_BASEM312_BASEM312_BASEM312_JOINTS140_reverse_tj_small_2: type fixed, parent BASEM9_BASEM312_BASEM312_BASEM312_BASEM312_BASEM312_BASEM312_BASEM312_JOINTS140_reverse_tj_in, child BASEM9_BASEM312_BASEM312_BASEM312_BASEM312_BASEM312_BASEM312_BASEM312_JOINTS140_reverse_tj_body, origin xyz=-0.057500000000000134 -0.0 0.036499999999999796 rpy=0.0 -1.5707963267949 0.0, axis 0 0 0
- added joint BASEM9_BASEM312_BASEM312_BASEM312_BASEM312_BASEM312_BASEM312_CONNECTORS145_reverse_ic_small_1: type fixed, parent BASEM9_BASEM312_BASEM312_BASEM312_BASEM312_BASEM312_BASEM312_CONNECTORS145_reverse_ic_body, child BASEM9_BASEM312_BASEM312_BASEM312_BASEM312_BASEM312_JOINTS141_reverse_tj_in, origin xyz=-0.0 -0.0 -0.0 rpy=0.0 0.0 0.0, axis 0 0 0
- added joint BASEM9_BASEM312_BASEM312_BASEM312_BASEM312_BASEM312_BASEM312_CONNECTORS145_reverse_ic_small_2: type fixed, parent BASEM9_BASEM312_BASEM312_BASEM312_BASEM312_BASEM312_BASEM312_CONNECTORS145_reverse_ic_in, child BASEM9_BASEM312_BASEM312_BASEM312_BASEM312_BASEM312_BASEM312_CONNECTORS145_reverse_ic_body, origin xyz=0.0 0.0 0.0073 rpy=0.0 0.0 3.141592653589793, axis 0 0 0
- added joint BASEM9_BASEM312_BASEM312_BASEM312_BASEM312_BASEM312_JOINTS141_reverse_tj_small_1: type revolute, parent BASEM9_BASEM312_BASEM312_BASEM312_BASEM312_BASEM312_JOINTS141_reverse_tj_body, child BASEM9_BASEM312_BASEM312_BASEM312_BASEM312_CONNECTORS146_reverse_ic_in, origin xyz=-0.0 -0.0 -0.0 rpy=0.0 0.0 0.0, axis 0 0 1, limit lower=-3.1416 upper=3.1416 effort=4.5 velocity=0.4
- added joint BASEM9_BASEM312_BASEM312_BASEM312_BASEM312_BASEM312_JOINTS141_reverse_tj_small_2: type fixed, parent BASEM9_BASEM312_BASEM312_BASEM312_BASEM312_BASEM312_JOINTS141_reverse_tj_in, child BASEM9_BASEM312_BASEM312_BASEM312_BASEM312_BASEM312_JOINTS141_reverse_tj_body, origin xyz=-0.057500000000000134 -0.0 0.036499999999999796 rpy=0.0 -1.5707963267949 0.0, axis 0 0 0
- added joint BASEM9_BASEM312_BASEM312_BASEM312_BASEM312_CONNECTORS146_reverse_ic_small_1: type fixed, parent BASEM9_BASEM312_BASEM312_BASEM312_BASEM312_CONNECTORS146_reverse_ic_body, child BASEM9_BASEM312_BASEM312_BASEM312_JOINTS142_reverse_tj_in, origin xyz=-0.0 -0.0 -0.0 rpy=0.0 0.0 0.0, axis 0 0 0
- added joint BASEM9_BASEM312_BASEM312_BASEM312_BASEM312_CONNECTORS146_reverse_ic_small_2: type fixed, parent BASEM9_BASEM312_BASEM312_BASEM312_BASEM312_CONNECTORS146_reverse_ic_in, child BASEM9_BASEM312_BASEM312_BASEM312_BASEM312_CONNECTORS146_reverse_ic_body, origin xyz=0.0 0.0 0.0073 rpy=0.0 0.0 3.141592653589793, axis 0 0 0
- added joint BASEM9_BASEM312_BASEM312_BASEM312_JOINTS142_reverse_tj_small_1: type revolute, parent BASEM9_BASEM312_BASEM312_BASEM312_JOINTS142_reverse_tj_body, child BASEM9_BASEM312_BASEM312_CONNECTORS147_reverse_CONNECTORS147_ic_in, origin xyz=-0.0 -0.0 -0.0 rpy=0.0 0.0 0.0, axis 0 0 1, limit lower=-3.1416 upper=3.1416 effort=4.5 velocity=0.4
- added joint BASEM9_BASEM312_BASEM312_BASEM312_JOINTS142_reverse_tj_small_2: type fixed, parent BASEM9_BASEM312_BASEM312_BASEM312_JOINTS142_reverse_tj_in, child BASEM9_BASEM312_BASEM312_BASEM312_JOINTS142_reverse_tj_body, origin xyz=-0.057500000000000134 -0.0 0.036499999999999796 rpy=0.0 -1.5707963267949 0.0, axis 0 0 0
- added joint BASEM9_BASEM312_BASEM312_CONNECTORS147_reverse_CONNECTORS147_ic_small_1: type fixed, parent BASEM9_BASEM312_BASEM312_CONNECTORS147_reverse_CONNECTORS147_ic_body, child BASEM9_BASEM312_ENDEFFECTORS4_ee_in, origin xyz=-0.0 -0.0 -0.0 rpy=0.0 0.0 0.0, axis 0 0 0
- added joint BASEM9_BASEM312_BASEM312_CONNECTORS147_reverse_CONNECTORS147_ic_small_2: type fixed, parent BASEM9_BASEM312_BASEM312_CONNECTORS147_reverse_CONNECTORS147_ic_in, child BASEM9_BASEM312_BASEM312_CONNECTORS147_reverse_CONNECTORS147_ic_body, origin xyz=-0.0 -0.0 0.0073 rpy=0.0 0.0 0.0, axis 0 0 0
- added joint BASEM9_BASEM312_ENDEFFECTORS4_ee_small: type fixed, parent BASEM9_BASEM312_ENDEFFECTORS4_ee_in, child BASEM9_BASEM312_ENDEFFECTORS4_ee_body, origin xyz=0 0 0 rpy=0 0 0, axis 0 0 0
